File: PLC4UNI_Board/PLC4UNI_Board.kicad_pcb (KiCad board)
At the start: 2 copper layers, 102.2 x 83 mm, 0 parts

Commit message: v2.1.0
Parts:
- added C1: 1uF, Capacitor_SMD:C_1206_3216Metric_Pad1.33x1.80mm_HandSolder, F.Cu at (301.0, 188.1)
- added C11: 100nF, Capacitor_SMD:C_0805_2012Metric, F.Cu at (362.8, 209.1)
- added C2: 22uF, Capacitor_SMD:C_1206_3216Metric, F.Cu at (359.6, 197.0)
- added C3: 100nF, Capacitor_SMD:C_0201_0603Metric, F.Cu at (360.2, 200.4)
- added C4: 22uF, Capacitor_SMD:C_1206_3216Metric_Pad1.33x1.80mm_HandSolder, F.Cu at (359.8, 193.7)
- added C5: 22uF, Capacitor_SMD:C_0805_2012Metric_Pad1.18x1.45mm_HandSolder, F.Cu at (356.6, 201.0)
- added C6: 22uF, Capacitor_SMD:C_0805_2012Metric_Pad1.18x1.45mm_HandSolder, F.Cu at (356.6, 204.1)
- added C7: 1uF, Capacitor_SMD:C_0805_2012Metric_Pad1.18x1.45mm_HandSolder, F.Cu at (380.0, 175.6)
- added C8: 100nF, Capacitor_SMD:C_0805_2012Metric, F.Cu at (379.8, 178.6)
- added C9: 100nF, Capacitor_SMD:C_0805_2012Metric_Pad1.18x1.45mm_HandSolder, F.Cu at (339.4, 204.6)
- added D1: 1N4001, Diode_THT:D_DO-41_SOD81_P10.16mm_Horizontal, F.Cu at (311.4, 208.2)
- added D2: SM712_SOT23, Package_TO_SOT_SMD:SOT-23, F.Cu at (355.5, 187.2)
- added D3: 1N4001, Diode_THT:D_DO-41_SOD81_P10.16mm_Horizontal, F.Cu at (362.4, 158.9)
- added D4: PTVS10VZ1USK, Diode_SMD:Nexperia_DSN1608-2_1.6x0.8mm, F.Cu at (342.6, 207.3)
- added D5: SMF24A, Diode_SMD:D_SMF, F.Cu at (374.7, 175.8)
- added ENTRADAS1: Screw_Terminal_01x18, TerminalBlock:TerminalBlock_MaiXu_MX126-5.0-18P_1x18_P5.00mm, F.Cu at (181.0, 103.5)
- added K1: G5Q-1, Relay_THT:Relay_SPDT_Omron-G5Q-1, F.Cu at (300.4, 203.6)
- added K2: G5Q-1, Relay_THT:Relay_SPDT_Omron-G5Q-1, F.Cu at (351.5, 154.3)
- added L1: 6.8uH_1.0A_4018, Inductor_SMD:L_APV_ANR6028, F.Cu at (352.9, 195.8)
- added Q10: TIP42, Package_TO_SOT_THT:TO-220-3_Vertical, F.Cu at (379.7, 148.1)
- added Q11: TIP42, Package_TO_SOT_THT:TO-220-3_Vertical, F.Cu at (388.6, 186.1)
- added Q4: TIP41, Package_TO_SOT_THT:TO-220-3_Vertical, F.Cu at (387.7, 171.1)
- added Q5: TIP41, Package_TO_SOT_THT:TO-220-3_Vertical, F.Cu at (375.1, 186.1)
- added Q6: TIP41, Package_TO_SOT_THT:TO-220-3_Vertical, F.Cu at (388.6, 198.2)
- added Q7: TIP41, Package_TO_SOT_THT:TO-220-3_Vertical, F.Cu at (301.2, 209.9)
- added Q8: TIP41, Package_TO_SOT_THT:TO-220-3_Vertical, F.Cu at (352.3, 160.7)
- added Q9: TIP42, Package_TO_SOT_THT:TO-220-3_Vertical, F.Cu at (375.1, 198.2)
- added R1: 10K, Resistor_SMD:R_0201_0603Metric, F.Cu at (309.2, 187.3)
- added R10: R_US, Resistor_SMD:R_0201_0603Metric, F.Cu at (373.1, 211.4)
- added R11: R_US, Resistor_SMD:R_0201_0603Metric, F.Cu at (373.1, 213.1)
- added R12: R_US, Resistor_SMD:R_0603_1608Metric, F.Cu at (387.4, 211.8)
- added R13: R_US, Resistor_SMD:R_0201_0603Metric, F.Cu at (390.6, 211.4)
- added R14: R_US, Resistor_SMD:R_0603_1608Metric, F.Cu at (339.0, 198.9)
- added R15: R_US, Resistor_SMD:R_0201_0603Metric, F.Cu at (342.2, 198.5)
- added R16: R_US, Resistor_SMD:R_0603_1608Metric, F.Cu at (378.5, 161.7)
- added R17: R_US, Resistor_SMD:R_0201_0603Metric, F.Cu at (381.7, 161.3)
- added R18: R_US, Resistor_SMD:R_0603_1608Metric, F.Cu at (351.0, 213.0)
- added R19: R_US, Resistor_SMD:R_0201_0603Metric, F.Cu at (354.3, 212.6)
- added R2: R_US, Resistor_SMD:R_0201_0603Metric, F.Cu at (360.2, 202.2)
- added R20: 120, Resistor_SMD:R_0603_1608Metric, F.Cu at (362.6, 211.8)
- added R21: 22K, Resistor_SMD:R_0603_1608Metric, F.Cu at (339.0, 207.4)
- added R22: R_US, Resistor_SMD:R_0201_0603Metric, F.Cu at (320.3, 211.2)
- added R23: R_US, Resistor_SMD:R_0201_0603Metric, F.Cu at (371.4, 161.9)
- added R24: 10K, Resistor_SMD:R_0603_1608Metric, F.Cu at (339.0, 209.9)
- added R25: 10k, Resistor_SMD:R_0603_1608Metric, F.Cu at (373.8, 178.7)
- added R26: 120, Resistor_SMD:R_0603_1608Metric, F.Cu at (351.0, 186.2)
- added R27: 120, Resistor_SMD:R_0603_1608Metric, F.Cu at (351.0, 188.7)
- added R3: R_US, Resistor_SMD:R_0201_0603Metric, F.Cu at (360.2, 203.9)
- added R31: 4.7k, Resistor_SMD:R_0603_1608Metric, F.Cu at (306.0, 187.7)
- added R32: 4.7k, Resistor_SMD:R_0603_1608Metric, F.Cu at (306.0, 190.2)
- added R4: R_US, Resistor_SMD:R_0201_0603Metric, F.Cu at (389.3, 161.3)
- added R5: R_US, Resistor_SMD:R_0201_0603Metric, F.Cu at (389.3, 163.1)
- added R6: R_US, Resistor_SMD:R_0201_0603Metric, F.Cu at (326.7, 198.5)
- added R7: R_US, Resistor_SMD:R_0201_0603Metric, F.Cu at (326.7, 200.3)
- added R8: R_US, Resistor_SMD:R_0201_0603Metric, F.Cu at (326.7, 208.2)
- added R9: R_US, Resistor_SMD:R_0201_0603Metric, F.Cu at (326.7, 209.9)
- added RS1: ~, TB'000H:RS485-MODULE-DEVO, F.Cu at (349.8, 184.2)
- added SALIDAS1: Screw_Terminal_01x18, TerminalBlock:TerminalBlock_MaiXu_MX126-5.0-18P_1x18_P5.00mm, F.Cu at (181.0, 178.0)
- added U1: ESP32-S3-WR-1, RF_Module:ESP32-S3-WROOM-1, F.Cu at (260.4, 143.0)
- added U10: TLP290, Package_SO:SOP-4_4.4x2.6mm_P1.27mm, F.Cu at (353.8, 209.6)
- added U11: TLP290, Package_SO:SOP-4_4.4x2.6mm_P1.27mm, F.Cu at (376.6, 202.3)
- added U12: TLP290, Package_SO:SOP-4_4.4x2.6mm_P1.27mm, F.Cu at (381.3, 152.2)
- added U13: TLP290, Package_SO:SOP-4_4.4x2.6mm_P1.27mm, F.Cu at (390.1, 190.2)
- added U14: TLP290, Package_SO:SOP-4_4.4x2.6mm_P1.27mm, F.Cu at (389.2, 175.2)
- added U15: TLP290, Package_SO:SOP-4_4.4x2.6mm_P1.27mm, F.Cu at (376.6, 190.2)
- added U16: TLP290, Package_SO:SOP-4_4.4x2.6mm_P1.27mm, F.Cu at (390.1, 202.3)
- added U17: TLP290, Package_SO:SOP-4_4.4x2.6mm_P1.27mm, F.Cu at (314.3, 212.4)
- added U18: TLP290, Package_SO:SOP-4_4.4x2.6mm_P1.27mm, F.Cu at (365.4, 163.1)
- added U19: ~, Package_SO:SOIC-8_5.3x5.3mm_P1.27mm, F.Cu at (377.0, 170.7)
- added U2: AP63203WU, Package_TO_SOT_SMD:TSOT-23-6, F.Cu at (351.6, 201.9)
- added U3: TLP290, Package_SO:SOP-4_4.4x2.6mm_P1.27mm, F.Cu at (392.8, 158.4)
- added U4: TLP290, Package_SO:SOP-4_4.4x2.6mm_P1.27mm, F.Cu at (330.2, 195.6)
- added U5: TLP290, Package_SO:SOP-4_4.4x2.6mm_P1.27mm, F.Cu at (330.2, 205.2)
- added U6: TLP290, Package_SO:SOP-4_4.4x2.6mm_P1.27mm, F.Cu at (376.6, 208.4)
- added U7: TLP290, Package_SO:SOP-4_4.4x2.6mm_P1.27mm, F.Cu at (390.1, 208.4)
- added U8: TLP290, Package_SO:SOP-4_4.4x2.6mm_P1.27mm, F.Cu at (341.8, 195.6)
- added U9: TLP290, Package_SO:SOP-4_4.4x2.6mm_P1.27mm, F.Cu at (381.3, 158.4)

Commit message: rs.v.2
Parts:
- removed D2: SM712_SOT23, Package_TO_SOT_SMD:SOT-23
- removed R26, R27: 120, Resistor_SMD:R_0603_1608Metric
- removed RS1: ~, TB'000H:RS485-MODULE-DEVO
- added J4: Conn_01x03, Connector_PinHeader_2.54mm:PinHeader_1x03_P2.54mm_Vertical, F.Cu at (1.79, 1.79)
- added U21: ~, ULTRARS485:Untitled, F.Cu at (254.5, 163.5)
- moved R4 261.5 mm to (128.3, 179.6)
- moved R5 261.5 mm to (128.3, 181.3)
- moved U3 261.5 mm to (131.9, 176.6)
- moved R10 260.2 mm to (116.7, 167.2)
- moved R11 260.2 mm to (116.7, 168.9)
- moved U6 260.2 mm to (120.2, 164.2)
- moved C2 251.1 mm to (110.2, 167.2)
- moved U2 251.1 mm to (102.2, 172.1)
- moved C3 251.1 mm to (110.8, 170.6)
- moved C5 251.1 mm to (107.2, 171.2)
- moved C6 251.1 mm to (107.2, 174.2)
- moved R2 251.1 mm to (110.8, 172.3)
- moved R3 251.1 mm to (110.8, 174.1)
- moved C4 251.1 mm to (110.4, 163.8)
- moved L1 251.1 mm to (103.5, 165.9)
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Connections:
- C8 pad 2: /0_10OUT/VOLTAGE_AOUTPUT -> /VOLTAGE_AOUTPUT
- D5 pad 1: /0_10OUT/VOLTAGE_AOUTPUT -> /VOLTAGE_AOUTPUT
- SALIDAS1 pad 1: /RS_485-A -> /NPN_O3
- SALIDAS1 pad 11: /NO2 -> /NO1
- SALIDAS1 pad 12: unconnected-(SALIDAS1-Pin_7-Pad12) -> /NC1
- SALIDAS1 pad 13: unconnected-(SALIDAS1-Pin_6-Pad13) -> /PNP_O3
- SALIDAS1 pad 14: /VOLTAGE_AOUTPUT -> /PNP_O2
- SALIDAS1 pad 15: GND2 -> /PNP_O1
- SALIDAS1 pad 16: /NPN_O1 -> GNDPWR
- SALIDAS1 pad 17: /NPN_O2 -> /RS_485-B
- SALIDAS1 pad 18: /NPN_O3 -> /RS_485-A
- SALIDAS1 pad 2: /RS_485-B -> /NPN_O2
- SALIDAS1 pad 3: GND2 -> /NPN_O1
- SALIDAS1 pad 4: /PNP_O1 -> GND2
- SALIDAS1 pad 5: /PNP_O2 -> /VOLTAGE_AOUTPUT
- SALIDAS1 pad 6: /PNP_O3 -> unconnected-(SALIDAS1-Pin_6-Pad6)
- SALIDAS1 pad 7: /NC1 -> unconnected-(SALIDAS1-Pin_7-Pad7)
- SALIDAS1 pad 8: /NO1 -> /NO2
- U1 pad 27: /PLC4UNI/UART_IN -> /mA_IN
- U1 pad 38: /mA_IN -> /PLC4UNI/UART_OUT
- U1 pad 39: /PLC4UNI/UART_OUT -> /PLC4UNI/UART_IN
- U19 pad 6: /0_10OUT/VOLTAGE_AOUTPUT -> /VOLTAGE_AOUTPUT
Routing:
- net /RS_485-A: track 0.00 -> 76.5 mm
- net GNDPWR: track 0.00 -> 76.3 mm
- net /RS_485-B: track 0.00 -> 71.5 mm
- net GND: track 0.00 -> 63.8 mm, vias 0 -> 6
- net +3.3V: track 0.00 -> 23.0 mm, vias 0 -> 1
- net /PLC4UNI/UART_IN: track 0.00 -> 16.1 mm, vias 0 -> 2
- net /PLC4UNI/UART_OUT: track 0.00 -> 13.0 mm, vias 0 -> 2
- net /0_10OUT/SEL: track 0.00 -> 8.38 mm
- net /VOLTAGE_AOUTPUT: track 0.00 -> 6.92 mm, vias 0 -> 2
- net Net-(U19-V5V): track 0.00 -> 3.11 mm
Other:
- copper layers 2 -> 4
