File: PLC4UNI_Board/PLC4UNI_Board.kicad_pcb (KiCad board)
At the start: 4 copper layers, 102.2 x 83 mm, 93 parts, among them J4 Conn_01x03, K1 G5Q-1, K2 G5Q-1, Q10 TIP42, Q11 TIP42, Q4 TIP41, Q5 TIP41, Q6 TIP41, Q7 TIP41, Q8 TIP41, Q9 TIP42, T1 IRF9310TRPBF, U1 ESP32-S3-WR-1, U10 TLP290, U11 TLP290, U12 TLP290, U13 TLP290, U14 TLP290, U15 TLP290, U16 TLP290, U17 TLP290, U18 TLP290, U2 AP63203WU, U3 TLP290, U4 TLP290, U5 TLP290, U6 TLP290, U7 TLP290, U8 TLP290, U9 TLP290

Commit message: main
Parts:
- removed J4: Conn_01x03, Connector_PinHeader_2.54mm:PinHeader_1x03_P2.54mm_Vertical
- added C10: 22PF, Capacitor_SMD:C_0603_1608Metric, F.Cu at (194.5, 133.0)
- added C17: 22PF, Capacitor_SMD:C_0603_1608Metric, F.Cu at (191.8, 141.0)
- added D8: ESDA5V3SC5, Package_TO_SOT_SMD:SOT-23-5, F.Cu at (199.4, 133.6)
- added R30: R5K1, Resistor_SMD:R_0201_0603Metric, F.Cu at (192.8, 134.8)
- added R33: R5K1, Resistor_SMD:R_0201_0603Metric, F.Cu at (191.0, 134.8)
- added R34: R5K1, Resistor_SMD:R_0201_0603Metric, F.Cu at (198.5, 136.6)
- added USB1: USB_C_Receptacle_USB2.0_14P, tipo-c-v:USB-C-TH_HX-TYPE-C-16P-180-LC-BH10.0-TYPE-C-VERTICAL, F.Cu at (191.2, 137.7)
- C3: footprint Capacitor_SMD:C_0201_0603Metric -> Resistor_SMD:R_0805_2012Metric
- C4: value 22uF -> 100pf; footprint Capacitor_SMD:C_1206_3216Metric_Pad1.33x1.80mm_HandSolder -> Resistor_SMD:R_0805_2012Metric
- D7: footprint Diode_THT:D_DO-41_SOD81_P10.16mm_Horizontal -> Diode_SMD:D_0603_1608Metric_Pad1.05x0.95mm_HandSolder
- JP1, JP2, JP3, U11, U12, U13, U14, U15, U16: moved to B.Cu
- L1: footprint Inductor_SMD:L_APV_ANR6028 -> Inductor_SMD:L_Changjiang_FNR5040S
- Q10, Q11, Q4, Q5, Q6, Q7, Q8, Q9: footprint Package_TO_SOT_THT:TO-220-3_Vertical -> Package_TO_SOT_SMD:TO-252-2
- R2: value R_US -> 30,9k; footprint Resistor_SMD:R_0201_0603Metric -> Resistor_SMD:R_0805_2012Metric
- R3: value R_US -> 62k
- moved T1 54.9 mm to (252.0, 122.2)
- moved D2 53.2 mm to (248.5, 129.3)
- moved R19 48.8 mm to (198.8, 109.7)
- moved U10 45.4 mm to (200.5, 112.9)
- moved JP1 43.8 mm to (245.0, 157.0)
- moved U20 42.0 mm to (242.6, 126.8)
- moved R18 40.6 mm to (202.9, 109.4)
- moved R17 37.1 mm to (204.6, 109.4)
- moved JP2 36.5 mm to (241.2, 157.0)
- moved R35 35.5 mm to (242.5, 136.8)
- moved R29 34.6 mm to (239.0, 133.5)
- moved R26 33.9 mm to (239.2, 135.5), turned to -90 degrees
- moved U9 33.6 mm to (206.4, 112.8)
- moved C13 32.8 mm to (241.4, 134.6)
- moved R27 32.5 mm to (240.8, 140.2)
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Connections:
- ENTRADAS1 pad 2: GND1 -> GND
- Q4 pad 3: GND -> GND3
- Q5 pad 3: GND -> GND3
- Q6 pad 3: GND -> GND3
- R17 pad 1: /PNP_MCU_1 -> /PNP_MCU_3
- SALIDAS1 pad 4: GND2 -> GND3
- SALIDAS1 pad 6: GND2 -> GND
- U1 pad 13: unconnected-(U1-USB_D--Pad13) -> /D-minus
- U1 pad 14: unconnected-(U1-USB_D+-Pad14) -> /D-plus
- U9 pad 3: /PNP_MCU_1 -> /PNP_MCU_3
Routing:
- net VCC: track 21.2 -> 306.1 mm, vias 0 -> 7
- net +3.3V: track 19.1 -> 192.1 mm, vias 0 -> 14
- net /PNP_MCU_3: track 0.00 -> 121.6 mm, vias 0 -> 2
- net GND: track 16.0 -> 116.6 mm, vias 0 -> 22
- net /PNP_MCU_4: track 0.00 -> 93.7 mm, vias 0 -> 3
- net /0_10OUT/SDA: track 0.00 -> 92.4 mm, vias 0 -> 6
- net /0_10OUT/SCLK: track 0.00 -> 86.1 mm, vias 0 -> 6
- net /D-minus: track 0.00 -> 81.9 mm, vias 0 -> 2
- net /D-plus: track 0.00 -> 78.3 mm, vias 0 -> 3
- net /mA_IN: track 7.00 -> 81.8 mm, vias 0 -> 4
- net GND2: track 0.00 -> 68.2 mm
- net /PLC4UNI/UART_IN: track 0.00 -> 66.2 mm, vias 0 -> 1
- net /PLC4UNI/UART_OUT: track 0.10 -> 64.2 mm, vias 0 -> 1
- net /NPN_MCU_2: track 0.00 -> 58.4 mm, vias 0 -> 2
- net /NPN_MCU_1: track 0.00 -> 56.6 mm, vias 0 -> 2
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- added copper zone on F.Cu, net GND
- removed copper zone on F.Cu, net GND2
Other:
- board text added: "22uF"

Commit message: main
Parts:
- added D10: 1N5819, Diode_SMD:D_0603_1608Metric_Pad1.05x0.95mm_HandSolder, F.Cu at (179.5, 130.0)
- added D9: 1N4007, Diode_SMD:D_0603_1608Metric_Pad1.05x0.95mm_HandSolder, F.Cu at (192.0, 128.2)
- added R36: 10K, Resistor_SMD:R_0603_1608Metric, F.Cu at (259.6, 125.6)
- added R37: 10K, Resistor_SMD:R_0603_1608Metric, F.Cu at (204.4, 122.9)
- added R38: 10K, Resistor_SMD:R_0603_1608Metric, F.Cu at (201.2, 121.8)
- added R39: 10K, Resistor_SMD:R_0603_1608Metric, F.Cu at (204.4, 128.4)
- added USB-SDCARD: USB_C_Receptacle_USB2.0_14P, tipo-c-v:USB-C-TH_HX-TYPE-C-16P-180-LC-BH10.0-TYPE-C-VERTICAL, F.Cu at (202.5, 125.3)
Connections:
- C2 pad 1: VCC -> /5vusb
- U1 pad 33: unconnected-(U1-IO40-Pad33) -> /DO
- U1 pad 34: unconnected-(U1-IO41-Pad34) -> /CS/CD
- U1 pad 35: unconnected-(U1-IO42-Pad35) -> /CMD/DI
- U2 pad 2: VCC -> /5vusb
- U2 pad 3: VCC -> /5vusb
- USB1 pad A4: VCC -> Net-(D9-A)
- USB1 pad A9: VCC -> Net-(D9-A)
- USB1 pad B4: VCC -> Net-(D9-A)
- USB1 pad B9: VCC -> Net-(D9-A)
Routing:
- net /DO: track 0.00 -> 153.6 mm, vias 0 -> 2
- net /CMD/DI: track 0.00 -> 98.0 mm, vias 0 -> 2
- net /CS/CD: track 0.00 -> 96.2 mm, vias 0 -> 1
- net /5vusb: track 0.00 -> 20.4 mm, vias 0 -> 2
- net +3.3V: track 192.1 -> 211.7 mm, vias 14 -> 19
- net Net-(D9-A): track 0.00 -> 18.9 mm
- net GND: track 116.6 -> 129.9 mm, vias 22 -> 26
- net Net-(USB2-GND-PadA1): track 0.00 -> 12.8 mm
- net /COM: track 52.7 -> 64.7 mm
- net Net-(USB2-VBUS-PadA4): track 0.00 -> 10.7 mm
- net /0_10OUT/SCLK: track 86.1 -> 92.6 mm
- net VCC: track 306.1 -> 302.8 mm, vias 7 -> 9
- net Net-(U19-V5V): track 14.6 -> 15.3 mm, vias 2 -> 3
