File: PLC4UNI_Board/untitled.kicad_sch (KiCad schematic)
At the start: 0 parts

Commit message: ok
Parts:
- added C1: 1uF, PCM_Capacitor_SMD_AKL:C_0603_1608Metric, symbol PCM_Capacitor_AKL:C_0603
- added R1: 10K, PCM_4ms_Resistor:R_0603, symbol Device:R_US
- added U1: ESP32-S3-WR-1, RF_Module:ESP32-S3-WROOM-1, symbol RF_Module:ESP32-S3-WROOM-1
Connections:
- new net: C1.1, R1.2, U1.3 (EN)
- new net +3.3V: R1.1, U1.2 (3V3)
- new net GND: C1.2, U1.1 (GND), U1.40 (GND), U1.41 (GND)
- new net UART_IN: U1.27 (IO0)
- new net UART_OUT: U1.39 (IO1)
Other:
- added sheet CT's CIRCUIT (CT's.kicad_sch)
- added sheet NPN_IN_1 (NPN.kicad_sch)
- added sheet NPN_IN_2 (NPN.kicad_sch)
- added sheet NPN_IN_3 (NPN.kicad_sch)
- added sheet NPN_IN_4 (NPN.kicad_sch)
- added sheet PNP_IN_1 (PNPI.kicad_sch)
- added sheet PNP_IN_2 (PNPI.kicad_sch)
- added sheet PNP_IN_3 (PNPI.kicad_sch)
- added sheet PNP_IN_4 (PNPI.kicad_sch)
- added sheet POWER_SUPPLY (PSU_sch.kicad_sch)

Commit message: v1.0.1
Other:
- added sheet NPN_OUT_1 (NPNO.kicad_sch)
- added sheet NPN_OUT_2 (NPNO.kicad_sch)
- added sheet NPN_OUT_3 (NPNO.kicad_sch)
- added sheet NPN_OUT_4 (NPNO.kicad_sch)
- added sheet PNP_OUT_1 (PNPO.kicad_sch)
- added sheet PNP_OUT_2 (PNPO.kicad_sch)
- added sheet PNP_OUT_3 (PNPO.kicad_sch)
- added sheet PNP_OUT_4 (PNPO.kicad_sch)
- added sheet RELAY_OUT_1 (RELO.kicad_sch)
- added sheet RELAY_OUT_2 (relo2.kicad_sch)
