File: PLC4UNI_Board/untitled.kicad_sch (KiCad schematic)
At the start: 3 parts, among them U1 ESP32-S3-WR-1

Commit message: main
Parts:
- C1: footprint PCM_Capacitor_SMD_AKL:C_0603_1608Metric -> Capacitor_SMD:C_1206_3216Metric_Pad1.33x1.80mm_HandSolder
- R1: footprint PCM_4ms_Resistor:R_0603 -> Resistor_SMD:R_0201_0603Metric
Connections:
- net RLO1: now reaches U1.10 (IO17)
- net RLO2: now reaches U1.11 (IO18)
Changed lines of the file:
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@@
+	(wire
+		(pts
+			(xy 190.5 92.71) (xy 186.69 92.71)
+		)
+		(stroke
+			(width 0)
+			(type default)
+		)
+	)
 	(wire
 		(pts
@@
 	(wire
 		(pts
+			(xy 190.5 95.25) (xy 186.69 95.25)
+		)
+		(stroke
+			(width 0)
+			(type default)
+		)
+	)
+	(wire
+		(pts
 			(xy 144.78 105.41) (xy 156.21 105.41)
 		)
@@
 		)
 	)
+	(hierarchical_label "RLO2"
+		(shape input)
+		(at 190.5 95.25 0)
+		(effects
+			(font
+				(size 1.27 1.27)
+			)
+			(justify left)
+		)
+	)
 	(hierarchical_label "UART_IN"
 		(shape input)
@@
 			)
 			(justify right)
+		)
+	)
+	(hierarchical_label "RLO1"
+		(shape input)
+		(at 190.5 92.71 0)
+		(effects
+			(font
+				(size 1.27 1.27)
+			)
+			(justify left)
 		)
 	)
@@
 			)
 		)
-		(property "Footprint" "PCM_Capacitor_SMD_AKL:C_0603_1608Metric"
+		(property "Footprint" "Capacitor_SMD:C_1206_3216Metric_Pad1.33x1.80mm_HandSolder"
 			(at 147.6248 85.09 0)
 			(effects
@@
 			)
 		)
-		(property "Footprint" "PCM_4ms_Resistor:R_0603"
+		(property "Footprint" "Resistor_SMD:R_0201_0603Metric"
 			(at 155.956 71.374 90)
 			(effects

Commit message: v2.1.0
Parts:
- added R31, R32: 4.7k, Resistor_SMD:R_0603_1608Metric, symbol Device:R
Connections:
- net +3.3V: now also R31.1, R32.1
- net AV_ADC: now reaches U1.23 (IO21)
- net SCLK: now reaches U1.28 (IO35)
- net SCLK: now also R31.2, R32.2
- net SDA: now reaches U1.29 (IO36)
- net SEL: now reaches U1.30 (IO37)
- net mA_READ: now reaches U1.38 (IO2)

Commit message: rs.v.2
Connections:
- net UART_IN: now also U1.39 (IO1); no longer U1.27 (IO0)
- net UART_OUT: now also U1.38 (IO2); no longer U1.39 (IO1)
- net mA_READ: now also U1.27 (IO0); no longer U1.38 (IO2)
Changed lines of the file:
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@@
-	(wire
-		(pts
-			(xy 149.86 95.25) (xy 156.21 95.25)
-		)
-		(stroke
-			(width 0)
-			(type default)
-		)
-	)
 	(wire
 		(pts
@@
 	(wire
 		(pts
-			(xy 149.86 92.71) (xy 156.21 92.71)
-		)
-		(stroke
-			(width 0)
-			(type default)
-		)
-	)
-	(wire
-		(pts
-			(xy 149.86 97.79) (xy 156.21 97.79)
-		)
-		(stroke
-			(width 0)
-			(type default)
-		)
-	)
-	(wire
-		(pts
 			(xy 186.69 105.41) (xy 205.74 105.41)
 		)
@@
 	(wire
 		(pts
+			(xy 144.78 95.25) (xy 156.21 95.25)
+		)
+		(stroke
+			(width 0)
+			(type default)
+		)
+	)
+	(wire
+		(pts
 			(xy 190.5 95.25) (xy 186.69 95.25)
 		)
@@
 	(wire
 		(pts
+			(xy 144.78 92.71) (xy 156.21 92.71)
+		)
+		(stroke
+			(width 0)
+			(type default)
+		)
+	)
+	(wire
+		(pts
 			(xy 148.59 77.47) (xy 154.94 77.47)
 		)
@@
 		(pts
 			(xy 144.78 128.27) (xy 156.21 128.27)
+		)
+		(stroke
+			(width 0)
+			(type default)
+		)
+	)
+	(wire
+		(pts
+			(xy 144.78 97.79) (xy 156.21 97.79)
 		)
 		(stroke
@@
 	(hierarchical_label "UART_OUT"
 		(shape bidirectional)
-		(at 149.86 95.25 180)
+		(at 144.78 97.79 180)
 		(effects
 			(font
@@
 	(hierarchical_label "UART_IN"
 		(shape bidirectional)
-		(at 149.86 92.71 180)
+		(at 144.78 95.25 180)
 		(effects
 			(font
@@
 	(hierarchical_label "mA_READ"
 		(shape bidirectional)
-		(at 149.86 97.79 180)
-		(effects
-			(font
+		(at 144.78 92.71 180)
+		(effects
+			(font

Commit message: v.3.0.0
Connections:
- net SCLK: no longer R32.2
- net SDA: now also R32.2
Changed lines of the file:
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@@
-	)
-	(junction
-		(at 213.36 105.41)
-		(diameter 0)
-		(color 0 0 0 0)
 	)
 	(junction
@@
 		(color 0 0 0 0)
 	)
+	(junction
+		(at 213.36 107.95)
+		(diameter 0)
+		(color 0 0 0 0)
+	)
 	(wire
 		(pts
@@
 	(wire
 		(pts
-			(xy 223.52 105.41) (xy 213.36 105.41)
-		)
-		(stroke
-			(width 0)
-			(type default)
-		)
-	)
-	(wire
-		(pts
 			(xy 154.94 74.93) (xy 154.94 77.47)
 		)
@@
 	(wire
 		(pts
-			(xy 213.36 104.14) (xy 213.36 105.41)
+			(xy 213.36 107.95) (xy 223.52 107.95)
 		)
 		(stroke
@@
 	(wire
 		(pts
-			(xy 186.69 107.95) (xy 223.52 107.95)
+			(xy 186.69 107.95) (xy 213.36 107.95)
 		)
 		(stroke
@@
 	(wire
 		(pts
+			(xy 213.36 104.14) (xy 213.36 107.95)
+		)
+		(stroke
+			(width 0)
+			(type default)
+		)
+	)
+	(wire
+		(pts
 			(xy 144.78 128.27) (xy 156.21 128.27)
 		)
@@
 	(wire
 		(pts
-			(xy 213.36 105.41) (xy 205.74 105.41)
-		)
-		(stroke
+			(xy 205.74 105.41) (xy 223.52 105.41)
+		)
+		(stroke

Commit message: main
Connections:
- net D-minus: now reaches U1.13 (USB_D-)
- net D-plus: now reaches U1.14 (USB_D+)
Changed lines of the file:
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@@
+	(wire
+		(pts
+			(xy 186.69 100.33) (xy 190.5 100.33)
+		)
+		(stroke
+			(width 0)
+			(type default)
+		)
+	)
 	(wire
 		(pts
 			(xy 144.78 115.57) (xy 156.21 115.57)
+		)
+		(stroke
+			(width 0)
+			(type default)
+		)
+	)
+	(wire
+		(pts
+			(xy 186.69 97.79) (xy 190.5 97.79)
 		)
 		(stroke
@@
 		)
 	)
+	(hierarchical_label "D-plus"
+		(shape input)
+		(at 190.5 100.33 0)
+		(effects
+			(font
+				(size 1.27 1.27)
+			)
+			(justify left)
+		)
+	)
 	(hierarchical_label "NPN_MCO_2"
 		(shape input)
@@
 		)
 	)
+	(hierarchical_label "D-minus"
+		(shape input)
+		(at 190.5 97.79 0)
+		(effects
+			(font
+				(size 1.27 1.27)
+			)
+			(justify left)
+		)
+	)

Commit message: main
Parts:
- added R37, R38, R39: 10K, Resistor_SMD:R_0603_1608Metric, symbol Device:R
Connections:
- net +3.3V: now also R37.1, R38.1, R39.1
- net DO: now reaches U1.33 (IO40)
- net DO: now also R37.2
- net CS/CD: now reaches U1.34 (IO41)
- net CS/CD: now also R38.2
- net CMD/DI: now reaches U1.35 (IO42)
- net CMD/DI: now also R39.2
