File: PLC4UNI_Board/ESP.kicad_sch (KiCad schematic)
At the start: 3 parts, among them U1 ESP32-S3-WR-1

Commit message: V1.0.2 PLC4UNI
Connections:
- net PNP_MCU_1: now also U1.38 (IO2); no longer U1.18 (IO10)
- net NPN_MC0_1: no longer names the net of U1.21 (IO13)
- net NPN_MCO_2: no longer names the net of U1.20 (IO12)
- net NPN_MCO_3: no longer names the net of U1.19 (IO11)
- net NPN_MCU_1: no longer names the net of U1.6 (IO6)
- net NPN_MCU_2: no longer names the net of U1.5 (IO5)
- net NPN_MCU_3: no longer names the net of U1.4 (IO4)
- net NPN_MCU_4: no longer names the net of U1.15 (IO3)
- net PNP_MCO_1: no longer names the net of U1.9 (IO16)
- net PNP_MCO_2: no longer names the net of U1.8 (IO15)
- net PNP_MCO_3: no longer names the net of U1.22 (IO14)
- net PNP_MCU_2: no longer names the net of U1.17 (IO9)
- net PNP_MCU_3: no longer names the net of U1.12 (IO8)
- net PNP_MCU_4: no longer names the net of U1.7 (IO7)
Other:
- removed sheet CT's CIRCUIT
- moved on the sheet: C1, R1, U1
