File: PLC4UNI_Board/NPN.kicad_sch (KiCad schematic)
At the start: 0 parts

Commit message: V1.0.2 PLC4UNI
Parts:
- added R4, R5: R_US, symbol Device:R_US
- added U3: TLP290, Package_SO:SOP-4_4.4x2.6mm_P1.27mm, symbol Isolator:TLP290
Connections:
- new net: R4.2, U3.1
- new net +3.3V: U3.4
- new net GND1: U3.2
- new net GND2: R5.2
- new net NPN_I1: R4.1
- new net NPN_MCU_1: R5.1, U3.3

Commit message: main
Parts:
- R4, R5: footprint (none) -> Resistor_SMD:R_0201_0603Metric
Connections:
- net GND2 is gone; now on net NPN_MCU_1: R5.2
- net +3.3V: now also R5.1; no longer U3.4
- net NPN_MCU_1: now also U3.4; no longer R5.1, U3.3
- new net GND: U3.3
Other:
- moved on the sheet: R5
Changed lines of the file:
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@@
 	(paper "A4")
 	(junction
-		(at 59.69 120.65)
+		(at 59.69 110.49)
 		(diameter 0)
 		(color 0 0 0 0)
@@
 	(wire
 		(pts
-			(xy 63.5 120.65) (xy 59.69 120.65)
+			(xy 67.31 110.49) (xy 59.69 110.49)
 		)
 		(stroke
@@
 	(wire
 		(pts
-			(xy 59.69 120.65) (xy 59.69 116.84)
+			(xy 33.02 116.84) (xy 44.45 116.84)
 		)
 		(stroke
@@
 	(wire
 		(pts
-			(xy 33.02 116.84) (xy 44.45 116.84)
+			(xy 59.69 120.65) (xy 59.69 116.84)
 		)
 		(stroke
@@
 	(hierarchical_label "NPN_MCU_1"
 		(shape input)
-		(at 63.5 120.65 0)
+		(at 67.31 110.49 0)
 		(effects
 			(font
@@
 	(symbol
 		(lib_id "power:+3.3V")
-		(at 59.69 110.49 0)
+		(at 59.69 102.87 0)
 		(unit 1)
 		(exclude_from_sim no)
@@
 		(fields_autoplaced yes)
 		(property "Reference" "#PWR05"
-			(at 59.69 114.3 0)
+			(at 59.69 106.68 0)
 			(effects
 				(font
@@
 		)
 		(property "Value" "+3.3V"
-			(at 59.69 105.41 0)
+			(at 59.69 97.79 0)
 			(effects
 				(font
@@
 		)
 		(property "Footprint" ""
-			(at 59.69 110.49 0)
+			(at 59.69 102.87 0)
 			(effects
 				(font
@@
 		)
 		(property "Datasheet" ""
-			(at 59.69 110.49 0)
+			(at 59.69 102.87 0)
 			(effects
 				(font
@@
 		)
 		(property "Description" "Power symbol creates a global label with name \"+3.3V\""
-			(at 59.69 110.49 0)
+			(at 59.69 102.87 0)
 			(effects
 				(font
@@
 		(on_board yes)
 		(dnp no)
-		(fields_autoplaced yes)
 		(property "Reference" "U3"
-			(at 52.07 105.41 0)
+			(at 50.038 105.156 0)
 			(effects
 				(font
@@
 		)
 		(property "Value" "TLP290"
-			(at 52.07 107.95 0)
+			(at 49.022 107.188 0)
 			(effects
 				(font
@@
 			)
 		)
-		(property "Footprint" ""
+		(property "Footprint" "Resistor_SMD:R_0201_0603Metric"
 			(at 40.894 110.744 90)
 			(effects
@@
 	(symbol
 		(lib_id "power:GND1")
-		(at 59.69 128.27 0)
+		(at 59.69 120.65 0)
 		(mirror y)
 		(unit 1)
@@
 		(dnp no)
 		(property "Reference" "#PWR06"
-			(at 59.69 134.62 0)
-			(effects
-				(font
-					(size 1.27 1.27)
-				)
-				(hide yes)
-			)
-		)
-		(property "Value" "GND2"
-			(at 59.69 131.826 0)
+			(at 59.69 127 0)
+			(effects
+				(font
+					(size 1.27 1.27)
+				)
+				(hide yes)
+			)
+		)
+		(property "Value" "GND"
+			(at 59.69 124.206 0)
 			(effects
 				(font
@@
 		)
 		(property "Footprint" ""
-			(at 59.69 128.27 0)
+			(at 59.69 120.65 0)
 			(effects
 				(font
@@
 		)
 		(property "Datasheet" ""
-			(at 59.69 128.27 0)
+			(at 59.69 120.65 0)
 			(effects
 				(font
@@
 		)
 		(property "Description" "Power symbol creates a global label with name \"GND1\" , ground"
-			(at 59.69 128.27 0)
+			(at 59.69 120.65 0)
 			(effects
 				(font
@@
 	(symbol
 		(lib_id "Device:R_US")
-		(at 59.69 124.46 0)
+		(at 59.69 106.68 0)
 		(unit 1)
 		(exclude_from_sim no)
@@
 		(dnp no)
 		(property "Reference" "R5"
-			(at 54.864 123.952 0)
+			(at 64.516 103.886 0)
 			(effects
 				(font
@@
 		)
 		(property "Value" "R_US"
-			(at 55.118 125.73 0)
-			(effects
-				(font
-					(size 1.27 1.27)
-				)
-			)
-		)
-		(property "Footprint" ""
-			(at 60.706 124.714 90)
+			(at 64.77 105.664 0)
+			(effects
+				(font
+					(size 1.27 1.27)
+				)
+			)
+		)
+		(property "Footprint" "Resistor_SMD:R_0201_0603Metric"
+			(at 60.706 106.934 90)
 			(effects
 				(font
@@
 		)
 		(property "Datasheet" "~"
-			(at 59.69 124.46 0)
+			(at 59.69 106.68 0)
 			(effects
 				(font
@@
 		)
 		(property "Description" "Resistor, US symbol"
-			(at 59.69 124.46 0)
-			(effects
-				(font
+			(at 59.69 106.68 0)
+			(effects
+				(font

Commit message: v.3.0.0
Connections:
- net GND1 renamed GND2
