File: PLC4UNI_Board/PNPI.kicad_sch (KiCad schematic)
At the start: 0 parts

Commit message: V1.0.2 PLC4UNI
Parts:
- added R12, R13: R_US, symbol Device:R_US
- added U7: TLP290, Package_SO:SOP-4_4.4x2.6mm_P1.27mm, symbol Isolator:TLP290
Connections:
- new net: R12.2, U7.2
- new net +3.3V: U7.4
- new net GND2: R13.2
- new net PNP_I1: R12.1
- new net PNP_MCU_1: R13.1, U7.3
- new net VCC: U7.1

Commit message: main
Parts:
- R12: footprint (none) -> Resistor_SMD:R_0603_1608Metric
- R13: footprint (none) -> Resistor_SMD:R_0201_0603Metric
Changed lines of the file:
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@@
 			)
 		)
-		(property "Footprint" ""
+		(property "Footprint" "Resistor_SMD:R_0603_1608Metric"
 			(at 43.434 85.344 90)
 			(effects
@@
 			)
 		)
-		(property "Footprint" ""
+		(property "Footprint" "Resistor_SMD:R_0201_0603Metric"
 			(at 69.596 90.424 90)
 			(effects

Commit message: v.3.0.0
Connections:
- net GND2 renamed GND
Changed lines of the file:
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@@
 			)
 		)
-		(property "Value" "GND2"
-			(at 68.58 104.14 0)
+		(property "Value" "GND"
+			(at 71.12 100.3299 0)
 			(effects
 				(font
 					(size 1.27 1.27)
 				)
+				(justify right)
 			)
 		)
