File: PLC4UNI_Board/NPNO.kicad_sch (KiCad schematic)
At the start: 0 parts

Commit message: V1.0.2 PLC4UNI
Parts:
- added Q4: TIP41, Package_TO_SOT_THT:TO-220-3_Vertical, symbol Transistor_BJT:TIP41
- added U14: TLP290, Package_SO:SOP-4_4.4x2.6mm_P1.27mm, symbol Isolator:TLP290
Connections:
- new net: Q4.1 (B), U14.3
- new net GND2: U14.2
- new net NPN_MCO_1: U14.1
- new net NPN_OUT_1: Q4.2 (C), U14.4
- new net VCC: Q4.3 (E)

Commit message: main
Connections:
- net VCC renamed GND
Changed lines of the file:
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@@
 	(wire
 		(pts
-			(xy 93.98 57.15) (xy 114.3 57.15)
+			(xy 93.98 57.15) (xy 99.06 57.15)
 		)
 		(stroke
@@
 	)
 	(symbol
+		(lib_id "power:GND2")
+		(at 99.06 57.15 0)
+		(unit 1)
+		(exclude_from_sim no)
+		(in_bom yes)
+		(on_board yes)
+		(dnp no)
+		(fields_autoplaced yes)
+		(property "Reference" "#PWR062"
+			(at 99.06 63.5 0)
+			(effects
+				(font
+					(size 1.27 1.27)
+				)
+				(hide yes)
+			)
+		)
+		(property "Value" "GND"
+			(at 99.06 62.23 0)
+			(effects
+				(font
+					(size 1.27 1.27)
+				)
+			)
+		)
+		(property "Footprint" ""
+			(at 99.06 57.15 0)
+			(effects
+				(font
+					(size 1.27 1.27)
+				)
+				(hide yes)
+			)
+		)
+		(property "Datasheet" ""
+			(at 99.06 57.15 0)
+			(effects
+				(font
+					(size 1.27 1.27)
+				)
+				(hide yes)
+			)
+		)
+		(property "Description" "Power symbol creates a global label with name \"GND2\" , ground"
+			(at 99.06 57.15 0)
+			(effects
+				(font
+					(size 1.27 1.27)
+				)
+				(hide yes)
+			)
+		)
+		(pin "1"
+		)
+		(instances
+			(project ""
+				(path "/3f95a48a-e63f-444a-b104-97d170acd68f/2020b834-9e04-4f06-8fda-b77ed6faff3c"
+					(reference "#PWR062")
+					(unit 1)
+				)
+				(path "/3f95a48a-e63f-444a-b104-97d170acd68f/4cd09166-bf28-4870-a4c5-3b89dcfb4047"
+					(reference "#PWR063")
+					(unit 1)
+				)
+				(path "/3f95a48a-e63f-444a-b104-97d170acd68f/bdcba0a6-fe9f-4879-9122-4774cf35b9dc"
+					(reference "#PWR064")
+					(unit 1)
+				)
+			)
+		)
+	)
+	(symbol
 		(lib_id "Isolator:TLP290")
 		(at 78.74 49.53 0)
@@
 					(unit 1)
 				)
-			)
-		)
-	)
-	(symbol
-		(lib_id "power:VCC")
-		(at 114.3 57.15 0)
-		(unit 1)
-		(exclude_from_sim no)
-		(in_bom yes)
-		(on_board yes)
-		(dnp no)
-		(fields_autoplaced yes)
-		(property "Reference" "#PWR045"
-			(at 114.3 60.96 0)
-			(effects
-				(font
-					(size 1.27 1.27)
-				)
-				(hide yes)
-			)
-		)
-		(property "Value" "VCC"
-			(at 114.3 52.07 0)
-			(effects
-				(font
-					(size 1.27 1.27)
-				)
-			)
-		)
-		(property "Footprint" ""
-			(at 114.3 57.15 0)
-			(effects
-				(font
-					(size 1.27 1.27)
-				)
-				(hide yes)
-			)
-		)
-		(property "Datasheet" ""
-			(at 114.3 57.15 0)
-			(effects
-				(font
-					(size 1.27 1.27)
-				)
-				(hide yes)
-			)
-		)
-		(property "Description" "Power symbol creates a global label with name \"VCC\""
-			(at 114.3 57.15 0)
-			(effects
-				(font
-					(size 1.27 1.27)
-				)
-				(hide yes)
-			)
-		)
-		(pin "1"
-		)
-		(instances
-			(project "PLC4UNI_Board"
-				(path "/3f95a48a-e63f-444a-b104-97d170acd68f/2020b834-9e04-4f06-8fda-b77ed6faff3c"
-					(reference "#PWR045")
-					(unit 1)
-				)
-				(path "/3f95a48a-e63f-444a-b104-97d170acd68f/4cd09166-bf28-4870-a4c5-3b89dcfb4047"
-					(reference "#PWR052")
-					(unit 1)
-				)
-				(path "/3f95a48a-e63f-444a-b104-97d170acd68f/bdcba0a6-fe9f-4879-9122-4774cf35b9dc"
-					(reference "#PWR054")
-					(unit 1)
-				)

Commit message: v.3.0.0
Connections:
- net GND2 is gone; now on net GND: U14.2
Changed lines of the file:
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@@
 			)
 		)
-		(property "Value" "GND2"
+		(property "Value" "GND"
 			(at 71.12 59.69 0)
 			(effects

Commit message: main
Parts:
- Q4: footprint Package_TO_SOT_THT:TO-220-3_Vertical -> Package_TO_SOT_SMD:TO-252-2
Connections:
- net GND: no longer Q4.3 (E)
- new net GND3: Q4.3 (E)
Changed lines of the file:
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@@
 			)
 		)
-		(property "Value" "GND"
+		(property "Value" "GND3"
 			(at 99.06 62.23 0)
 			(effects
@@
 			)
 		)
-		(property "Footprint" "Package_TO_SOT_THT:TO-220-3_Vertical"
+		(property "Footprint" "Package_TO_SOT_SMD:TO-252-2"
 			(at 97.79 53.975 0)
 			(effects
