File: PLC4UNI_Board/PLC4UNI_Board.kicad_sch (KiCad schematic)
At the start: 8 parts, among them J1 Screw_Terminal_01x04, J2 Screw_Terminal_01x05, J3 Screw_Terminal_01x02, J4 Screw_Terminal_01x03, J5 Screw_Terminal_01x03, J6 Screw_Terminal_01x04, J7 Screw_Terminal_01x06, J8 Screw_Terminal_01x02

Commit message: ok
Parts:
- removed J2: Screw_Terminal_01x05, symbol Connector:Screw_Terminal_01x05
- removed J3: Screw_Terminal_01x02, symbol Connector:Screw_Terminal_01x02
- removed J4, J5: Screw_Terminal_01x03, symbol Connector:Screw_Terminal_01x03
- removed J6: Screw_Terminal_01x04, symbol Connector:Screw_Terminal_01x04
- removed J7: Screw_Terminal_01x06, symbol Connector:Screw_Terminal_01x06
- added J10: RLY_OUT, symbol Connector:Screw_Terminal_01x03
- added J11: RLY2_OUT, symbol Connector:Screw_Terminal_01x02
- added J12: 0-10_AC, symbol Connector:Screw_Terminal_01x02
- added J2: NPN_IN, symbol Connector:Screw_Terminal_01x04
- added J3: AN_IN_OUT, symbol Connector:Screw_Terminal_01x04
- added J4: ANA_V_0-10, symbol Connector:Screw_Terminal_01x02
- added J5: CT_TC, symbol Connector:Screw_Terminal_01x02
- added J6: RS_485, symbol Connector:Screw_Terminal_01x03
- added J7: PNP_OUT, symbol Connector:Screw_Terminal_01x04
- added J9: PNP_IN, symbol Connector:Screw_Terminal_01x04
- J1: value Screw_Terminal_01x04 -> NPN_OUT
- J8: value Screw_Terminal_01x02 -> 24_V_DC
Connections:
- net GND: no longer J1.4 (Pin_4)
- net PLC4UNI/32V_ana: no longer names the net of J1.1 (Pin_1)
- net PLC4UNI/ANALOG_0-10v: no longer names the net of J1.2 (Pin_2)
- net PLC4UNI/ANALOG_4-20mA: no longer names the net of J1.3 (Pin_3)
Other:
- sheet PLC4UNI ports: added none; removed 32V_ana, ANALOGOUT_0-10v, ANALOGOUT_4-20mA, ANALOG_0-10v, ANALOG_4-20mA, COM_RLY1, COM_RLY2, DIGITAL_IN1, DIGITAL_IN2, INPUTNPN1, INPUTNPN2, INPUTPNP1, INPUTPNP2, NC_RLY1, NC_RLY2, NO_RLY1, NO_RLY2, NPN_I1, NPN_I2, PNP_I1, PNP_I2, RS_485-A, RS_485-B
- moved on the sheet: J8

Commit message: v.1.0.1
Parts:
- J1, J2, J9: footprint (none) -> tb-002H:TE_796683-4
- J10, J6: footprint (none) -> TB'000H:tb
- J11, J12, J4, J5, J8: footprint (none) -> tb-003H:EBBA-02-C-SS-BU
- J3, J7: footprint (none) -> TB'000H:terminal block
Changed lines of the file:
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@@
 			)
 		)
-		(property "Footprint" ""
+		(property "Footprint" "tb-003H:EBBA-02-C-SS-BU"
 			(at 132.08 58.42 0)
 			(effects
@@
 			)
 		)
-		(property "Footprint" ""
+		(property "Footprint" "TB'000H:terminal block"
 			(at 109.22 90.17 0)
 			(effects
@@
 			)
 		)
-		(property "Footprint" ""
+		(property "Footprint" "tb-003H:EBBA-02-C-SS-BU"
 			(at 182.88 124.46 0)
 			(effects
@@
 			)
 		)
-		(property "Footprint" ""
+		(property "Footprint" "tb-003H:EBBA-02-C-SS-BU"
 			(at 109.22 116.84 0)
 			(effects
@@
 			)
 		)
-		(property "Footprint" ""
+		(property "Footprint" "TB'000H:terminal block"
 			(at 182.88 80.01 0)
 			(effects
@@
 			)
 		)
-		(property "Footprint" ""
+		(property "Footprint" "TB'000H:tb"
 			(at 109.22 110.49 0)
 			(effects
@@
 			)
 		)
-		(property "Footprint" ""
+		(property "Footprint" "tb-002H:TE_796683-4"
 			(at 182.88 102.87 0)
 			(effects
@@
 			)
 		)
-		(property "Footprint" ""
+		(property "Footprint" "tb-002H:TE_796683-4"
 			(at 182.88 91.44 0)
 			(effects
@@
 			)
 		)
-		(property "Footprint" ""
+		(property "Footprint" "tb-003H:EBBA-02-C-SS-BU"
 			(at 182.88 118.11 0)
 			(effects
@@
 			)
 		)
-		(property "Footprint" ""
+		(property "Footprint" "tb-002H:TE_796683-4"
 			(at 109.22 101.6 0)
 			(effects
@@
 			)
 		)
-		(property "Footprint" ""
+		(property "Footprint" "tb-003H:EBBA-02-C-SS-BU"
 			(at 182.88 111.76 0)
 			(effects
@@
 			)
 		)
-		(property "Footprint" ""
+		(property "Footprint" "TB'000H:tb"
 			(at 109.22 77.47 0)
 			(effects
@@
 				(font
 					(size 1.27 1.27)
-				)
-				(hide yes)
+					(italic yes)
+				)
+				(hide yes)

Commit message: V1.0.2 PLC4UNI
Parts:
- removed J1: NPN_OUT, tb-002H:TE_796683-4, symbol Connector:Screw_Terminal_01x04
- removed J10: RLY_OUT, TB'000H:tb, symbol Connector:Screw_Terminal_01x03
- removed J12: 0-10_AC, tb-003H:EBBA-02-C-SS-BU, symbol Connector:Screw_Terminal_01x02
- removed J2: NPN_IN, tb-002H:TE_796683-4, symbol Connector:Screw_Terminal_01x04
- removed J3: AN_IN_OUT, TB'000H:terminal block, symbol Connector:Screw_Terminal_01x04
- removed J4: ANA_V_0-10, tb-003H:EBBA-02-C-SS-BU, symbol Connector:Screw_Terminal_01x02
- removed J5: CT_TC, tb-003H:EBBA-02-C-SS-BU, symbol Connector:Screw_Terminal_01x02
- removed J6: RS_485, TB'000H:tb, symbol Connector:Screw_Terminal_01x03
- removed J7: PNP_OUT, TB'000H:terminal block, symbol Connector:Screw_Terminal_01x04
- removed J8: 24_V_DC, tb-003H:EBBA-02-C-SS-BU, symbol Connector:Screw_Terminal_01x02
- removed J9: PNP_IN, tb-002H:TE_796683-4, symbol Connector:Screw_Terminal_01x04
- added J1, J4, J6: Screw_Terminal_01x18, symbol Connector:Screw_Terminal_01x18
Connections:
- net GND: now also J1.17 (Pin_17), J1.5 (Pin_5), J6.17 (Pin_17), J6.5 (Pin_5)
- net VCC: now also J1.18 (Pin_18), J6.18 (Pin_18)
- new net GND2: J4.16 (Pin_16)
- new net NPN_I1: J1.14 (Pin_14), J6.14 (Pin_14)
- new net NPN_I2: J1.13 (Pin_13), J6.13 (Pin_13)
- new net NPN_I3: J1.12 (Pin_12), J6.12 (Pin_12)
- new net NPN_I4: J1.11 (Pin_11), J6.11 (Pin_11)
- new net NPN_O1: J4.3 (Pin_3)
- new net NPN_O2: J4.2 (Pin_2)
- new net NPN_O3: J4.1 (Pin_1)
- new net PNP_I1: J1.9 (Pin_9), J6.9 (Pin_9)
- new net PNP_I2: J1.8 (Pin_8), J6.8 (Pin_8)
- new net PNP_I3: J1.7 (Pin_7), J6.7 (Pin_7)
- new net PNP_I4: J1.6 (Pin_6), J6.6 (Pin_6)
- new net PNP_O1: J4.15 (Pin_15)
- new net PNP_O2: J4.14 (Pin_14)
- new net PNP_O3: J4.13 (Pin_13)
- new net RS_485-A: J4.18 (Pin_18)
- new net RS_485-B: J4.17 (Pin_17)
Other:
- added sheet NPN_IN_1 (NPN.kicad_sch)
- added sheet NPN_IN_2 (NPN.kicad_sch)
- added sheet NPN_IN_3 (NPN.kicad_sch)
- added sheet NPN_IN_4 (NPN.kicad_sch)
- added sheet NPN_OUT_1 (NPNO.kicad_sch)
- added sheet NPN_OUT_3 (NPNO.kicad_sch)
- added sheet PNP_IN_1 (PNPI.kicad_sch)
- added sheet PNP_IN_2 (PNPI.kicad_sch)
- added sheet PNP_IN_3 (PNPI.kicad_sch)
- added sheet PNP_IN_4 (PNPI.kicad_sch)
- added sheet PNP_OUT_1 (PNPO.kicad_sch)
- added sheet PNP_OUT_2 (PNPO.kicad_sch)
- added sheet PNP_OUT_3 (PNPO.kicad_sch)
- added sheet POWER_SUPPLY (PSU_sch.kicad_sch)
- added sheet RS485 (RS485.kicad_sch)
- sheet PLC4UNI ports: added NPN_MC0_1, NPN_MCO_2, NPN_MCO_3, NPN_MCU_1, NPN_MCU_2, NPN_MCU_3, NPN_MCU_4, PNP_MCO_1, PNP_MCO_2, PNP_MCO_3, PNP_MCU_1, PNP_MCU_2, PNP_MCU_3, PNP_MCU_4, RS_485-A, RS_485-B, UART_IN, UART_OUT; removed none
- note added: "0-10_VAC"
- note added: "0-10v in 2 PINS"
- note added: "010oUT 2PINS"
- note added: "24VDC 2 PINS"
- note added: "4-20mA 2 PINS"
- note added: "420oUT 2PINS"
- note added: "CT_TC"
- note added: "NPN_OUT 3PINES"
- note added: "NPN__IN 4 PINS"
- note added: "PNP_OUT 3PINES"
- note added: "PNP__IN 4 PINS"
- note added: "RLY 2PINS"
- note added: "RLY 3PINES"
- note added: "RS485 3PINES"
- moved on the sheet: J11

Commit message: main
Parts:
- removed J1: Screw_Terminal_01x18, symbol Connector:Screw_Terminal_01x18
- removed J11: RLY2_OUT, tb-003H:EBBA-02-C-SS-BU, symbol Connector:Screw_Terminal_01x02
- ENTRADAS1: renamed from J6; footprint (none) -> TerminalBlock:TerminalBlock_MaiXu_MX126-5.0-18P_1x18_P5.00mm
- SALIDAS1: renamed from J4; footprint (none) -> TerminalBlock:TerminalBlock_MaiXu_MX126-5.0-18P_1x18_P5.00mm
Connections:
- net GND: now also ENTRADAS1.14 (Pin_5), ENTRADAS1.2 (Pin_17); no longer ENTRADAS1.17 (Pin_17), ENTRADAS1.5 (Pin_5)
- net GND2: now also SALIDAS1.3 (Pin_16); no longer SALIDAS1.16 (Pin_16)
- net NPN_I1: now also ENTRADAS1.5 (Pin_14); no longer ENTRADAS1.14 (Pin_14)
- net NPN_I2: now also ENTRADAS1.6 (Pin_13); no longer ENTRADAS1.13 (Pin_13)
- net NPN_I3: now also ENTRADAS1.7 (Pin_12); no longer ENTRADAS1.12 (Pin_12)
- net NPN_I4: now also ENTRADAS1.8 (Pin_11); no longer ENTRADAS1.11 (Pin_11)
- net NPN_O1: now also SALIDAS1.16 (Pin_3); no longer SALIDAS1.3 (Pin_3)
- net NPN_O2: now also SALIDAS1.17 (Pin_2); no longer SALIDAS1.2 (Pin_2)
- net NPN_O3: now also SALIDAS1.18 (Pin_1); no longer SALIDAS1.1 (Pin_1)
- net PNP_I1: now also ENTRADAS1.10 (Pin_9); no longer ENTRADAS1.9 (Pin_9)
- net PNP_I2: now also ENTRADAS1.11 (Pin_8); no longer ENTRADAS1.8 (Pin_8)
- net PNP_I3: now also ENTRADAS1.12 (Pin_7); no longer ENTRADAS1.7 (Pin_7)
- net PNP_I4: now also ENTRADAS1.13 (Pin_6); no longer ENTRADAS1.6 (Pin_6)
- net PNP_O1: now also SALIDAS1.4 (Pin_15); no longer SALIDAS1.15 (Pin_15)
- net PNP_O2: now also SALIDAS1.5 (Pin_14); no longer SALIDAS1.14 (Pin_14)
- net PNP_O3: now also SALIDAS1.6 (Pin_13); no longer SALIDAS1.13 (Pin_13)
- net RS_485-A: now also SALIDAS1.1 (Pin_18); no longer SALIDAS1.18 (Pin_18)
- net RS_485-B: now also SALIDAS1.2 (Pin_17); no longer SALIDAS1.17 (Pin_17)
- net VCC: now also ENTRADAS1.1 (Pin_18); no longer ENTRADAS1.18 (Pin_18)
- net COM: now reaches SALIDAS1.10 (Pin_9)
- net COM: now also SALIDAS1.9 (Pin_10)
- net NO2: now reaches SALIDAS1.11 (Pin_8)
- net NC1: now reaches SALIDAS1.7 (Pin_12)
- net NO1: now reaches SALIDAS1.8 (Pin_11)
Other:
- added sheet 4?20mA (420.kicad_sch)
- added sheet RLY_OUT_1 (RLY1.kicad_sch)
- added sheet RLY_OUT_2 (RLY1.kicad_sch)
- sheet PLC4UNI ports: added RLO1, RLO2; removed none
- moved on the sheet: SALIDAS1

Commit message: v2.1.0
Connections:
- net GND: now also ENTRADAS1.4 (Pin_15)
- net GND2: now also SALIDAS1.15 (Pin_4)
- net mA_IN: now reaches ENTRADAS1.3 (Pin_16)
- net AV_IN: now reaches ENTRADAS1.9 (Pin_10)
- net VOLTAGE_AOUTPUT: now reaches SALIDAS1.14 (Pin_5)
Other:
- sheet 4?20mA renamed IN4?20mA
- added sheet 010V (VA.kicad_sch)
- added sheet 0_10OUT (0_10VOUT.kicad_sch)
- sheet IN4?20mA ports: added mA_IN, mA_READ; removed none
- sheet PLC4UNI ports: added AV_ADC, SCLK, SDA, SEL, mA_READ; removed RS_485-A, RS_485-B
- moved on the sheet: ENTRADAS1, SALIDAS1

Commit message: rs.v.2
Connections:
- net GND2: now also SALIDAS1.4 (Pin_4); no longer SALIDAS1.15 (Pin_4), SALIDAS1.3 (Pin_16)
- net NC1: now also SALIDAS1.12 (7); no longer SALIDAS1.7 (Pin_12)
- net NO1: now also SALIDAS1.11 (Pin_11); no longer SALIDAS1.8 (Pin_11)
- net NO2: now also SALIDAS1.8 (Pin_8); no longer SALIDAS1.11 (Pin_8)
- net NPN_O1: now also SALIDAS1.3 (Pin_3); no longer SALIDAS1.16 (Pin_3)
- net NPN_O2: now also SALIDAS1.2 (Pin_2); no longer SALIDAS1.17 (Pin_2)
- net NPN_O3: now also SALIDAS1.1; no longer SALIDAS1.18 (Pin_1)
- net PNP_O1: now also SALIDAS1.15 (Pin_15); no longer SALIDAS1.4 (Pin_15)
- net PNP_O2: now also SALIDAS1.14; no longer SALIDAS1.5 (Pin_14)
- net PNP_O3: now also SALIDAS1.13 (Pin_13); no longer SALIDAS1.6 (Pin_13)
- net RS_485-A: now also SALIDAS1.18 (Pin_18); no longer SALIDAS1.1 (Pin_18)
- net RS_485-B: now also SALIDAS1.17 (Pin_17); no longer SALIDAS1.2 (Pin_17)
- net VOLTAGE_AOUTPUT: now also SALIDAS1.5 (Pin_5); no longer SALIDAS1.14 (Pin_5)
- new net GNDPWR: SALIDAS1.16
Other:
- sheet RS485: file RS485.kicad_sch -> RS_MOD_PRO.kicad_sch
Changed lines of the file:
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@@
 	(wire
 		(pts
+			(xy 31.75 74.93) (xy 34.925 74.93)
+		)
+		(stroke
+			(width 0)
+			(type default)
+		)
+	)
+	(wire
+		(pts
 			(xy 55.88 118.11) (xy 54.61 118.11)
 		)
@@
 	(wire
 		(pts
-			(xy 74.93 144.78) (xy 88.9 144.78)
-		)
-		(stroke
-			(width 0)
-			(type default)
-		)
-	)
-	(wire
-		(pts
 			(xy 171.45 39.37) (xy 168.91 39.37)
 		)
@@
 	(wire
 		(pts
-			(xy 74.93 149.86) (xy 76.2 149.86)
+			(xy 90.17 144.78) (xy 90.17 146.05)
 		)
 		(stroke
@@
 	(wire
 		(pts
-			(xy 33.655 74.93) (xy 34.29 74.93)
+			(xy 74.93 149.86) (xy 76.2 149.86)
 		)
 		(stroke
@@
 	(wire
 		(pts
+			(xy 74.93 144.78) (xy 90.17 144.78)
+		)
+		(stroke
+			(width 0)
+			(type default)
+		)
+	)
+	(wire
+		(pts
 			(xy 74.93 180.34) (xy 76.2 180.34)
 		)
@@
 	(hierarchical_label "VOLTAGE_AOUTPUT"
 		(shape bidirectional)
-		(at 33.655 74.93 180)
+		(at 31.75 74.93 180)
 		(effects
 			(font
@@
 	)
 	(symbol
-		(lib_id "power:GND")
-		(at 88.9 144.78 0)
-		(unit 1)
-		(exclude_from_sim no)
-		(in_bom yes)
-		(on_board yes)
-		(dnp no)
-		(property "Reference" "#PWR037"
-			(at 88.9 151.13 0)
-			(effects
-				(font
-					(size 1.27 1.27)
-				)
-				(hide yes)
-			)
-		)
-		(property "Value" "GND2"
-			(at 89.154 148.59 0)
-			(effects
-				(font
-					(size 1.27 1.27)
-				)
-			)
-		)
-		(property "Footprint" ""
-			(at 88.9 144.78 0)
-			(effects
-				(font
-					(size 1.27 1.27)
-				)
-				(hide yes)
-			)
-		)
-		(property "Datasheet" ""
-			(at 88.9 144.78 0)
-			(effects
-				(font
-					(size 1.27 1.27)
-				)
-				(hide yes)
-			)
-		)
-		(property "Description" "Power symbol creates a global label with name \"GND\" , ground"
-			(at 88.9 144.78 0)
-			(effects
-				(font
-					(size 1.27 1.27)
-				)
-				(hide yes)
-			)
-		)
-		(pin "1"
-		)
-		(instances
-			(project "PLC4UNI_Board"
-				(path "/3f95a48a-e63f-444a-b104-97d170acd68f"
-					(reference "#PWR037")
-					(unit 1)
-				)
-			)
-		)
-	)
-	(symbol
 		(lib_id "Connector:Screw_Terminal_01x18")
 		(at 118.11 166.37 0)
@@
 		(pin "4"
 		)
-		(pin "1"
+		(pin "18"
 		)
 		(pin "2"
@@
 		(pin "3"
 		)
-		(pin "14"
+		(pin "5"
 		)
 		(pin "17"
@@
 		(pin "13"
 		)
-		(pin "5"
+		(pin "14"
 		)
 		(pin "9"
@@
 		(pin "16"
 		)
-		(pin "18"
+		(pin "1"
 		)
 		(pin "10"
@@
 		)
 	)
+	(symbol
+		(lib_id "power:GNDPWR")
+		(at 90.17 146.05 0)
+		(unit 1)
+		(exclude_from_sim no)
+		(in_bom yes)
+		(on_board yes)
+		(dnp no)
+		(fields_autoplaced yes)
+		(property "Reference" "#PWR059"
+			(at 90.17 151.13 0)
+			(effects
+				(font
+					(size 1.27 1.27)
+				)
+				(hide yes)
+			)
+		)
+		(property "Value" "GNDPWR"
+			(at 90.043 149.86 0)
+			(effects
+				(font
+					(size 1.27 1.27)
+				)
+			)
+		)
+		(property "Footprint" ""
+			(at 90.17 147.32 0)
+			(effects
+				(font
+					(size 1.27 1.27)
+				)
+				(hide yes)
+			)
+		)
+		(property "Datasheet" ""
+			(at 90.17 147.32 0)
+			(effects
+				(font
+					(size 1.27 1.27)
+				)
+				(hide yes)
+			)
+		)
+		(property "Description" "Power symbol creates a global label with name \"GNDPWR\" , global ground"
+			(at 90.17 146.05 0)
+			(effects
+				(font
+					(size 1.27 1.27)
+				)
+				(hide yes)
+			)
+		)
+		(pin "1"
+		)
+		(instances
+			(project "PLC4UNI_Board"
+				(path "/3f95a48a-e63f-444a-b104-97d170acd68f"
+					(reference "#PWR059")
+					(unit 1)
+				)
+			)
+		)
+	)
 	(sheet
 		(at 34.4131 113.665)
@@
 			)
 		)
-		(property "Sheetfile" "RS485.kicad_sch"
+		(property "Sheetfile" "RS_MOD_PRO.kicad_sch"
 			(at 34.29 50.1146 0)
 			(effects

Commit message: v.3.0.0
Connections:
- net GND: no longer ENTRADAS1.2 (Pin_17), ENTRADAS1.4 (Pin_15)
- net GND2: now also ENTRADAS1.4 (Pin_15), SALIDAS1.6 (Pin_6)
- net mA_AOUTPUT+: now reaches SALIDAS1.7 (Pin_7)
- new net GND1: ENTRADAS1.2 (Pin_17)
Other:
- added sheet mA_INTERFAZ_OUT (mA_INTERFAZ.kicad_sch)

Commit message: main
Connections:
- net GND1 is gone; now on net GND: ENTRADAS1.2 (Pin_17)
- net GND: now also SALIDAS1.6 (Pin_6)
- net GND2: no longer SALIDAS1.4 (Pin_4), SALIDAS1.6 (Pin_6)
- new net GND3: SALIDAS1.4 (Pin_4)
Other:
- added sheet usb-c (usb.kicad_sch)
- sheet PLC4UNI ports: added D-minus, D-plus; removed none
- sheet POWER_SUPPLY ports: added 5vusb; removed none
