File: PLC4UNI_Board/PLC4UNI_Board.kicad_sch (KiCad schematic)
At the start: 2 parts

Commit message: main
Other:
- added sheet SD (SDC.kicad_sch)
- sheet PLC4UNI ports: added CMD/DI, CS/CD, DO; removed none
Changed lines of the file:
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@@
 	(wire
 		(pts
+			(xy 127 68.58) (xy 125.73 68.58)
+		)
+		(stroke
+			(width 0)
+			(type default)
+		)
+	)
+	(wire
+		(pts
+			(xy 127 71.12) (xy 125.73 71.12)
+		)
+		(stroke
+			(width 0)
+			(type default)
+		)
+	)
+	(wire
+		(pts
 			(xy 57.15 41.91) (xy 64.77 41.91)
 		)
@@
 	(wire
 		(pts
+			(xy 166.37 137.16) (xy 168.275 137.16)
+		)
+		(stroke
+			(width 0)
+			(type default)
+		)
+	)
+	(wire
+		(pts
 			(xy 55.88 76.2) (xy 64.77 76.2)
 		)
@@
 	(wire
 		(pts
+			(xy 166.37 139.7) (xy 168.275 139.7)
+		)
+		(stroke
+			(width 0)
+			(type default)
+		)
+	)
+	(wire
+		(pts
 			(xy 109.22 166.37) (xy 113.03 166.37)
 		)
@@
 	(wire
 		(pts
+			(xy 127 66.04) (xy 125.73 66.04)
+		)
+		(stroke
+			(width 0)
+			(type default)
+		)
+	)
+	(wire
+		(pts
 			(xy 74.93 147.32) (xy 76.2 147.32)
 		)
@@
 	(wire
 		(pts
+			(xy 166.37 144.78) (xy 168.275 144.78)
+		)
+		(stroke
+			(width 0)
+			(type default)
+		)
+	)
+	(wire
+		(pts
 			(xy 76.2 165.1) (xy 74.93 165.1)
 		)
@@
 	(wire
 		(pts
+			(xy 166.37 142.24) (xy 168.275 142.24)
+		)
+		(stroke
+			(width 0)
+			(type default)
+		)
+	)
+	(wire
+		(pts
 			(xy 199.39 53.34) (xy 198.12 53.34)
 		)
@@
 		)
 	)
+	(hierarchical_label "CMD{slash}DI"
+		(shape input)
+		(at 166.37 137.16 180)
+		(effects
+			(font
+				(size 1.27 1.27)
+			)
+			(justify right)
+		)
+	)
 	(hierarchical_label "COM"
 		(shape bidirectional)
@@
 		)
 	)
+	(hierarchical_label "SCLK"
+		(shape input)
+		(at 166.37 144.78 180)
+		(effects
+			(font
+				(size 1.27 1.27)
+			)
+			(justify right)
+		)
+	)
 	(hierarchical_label "PNP_O3"
 		(shape input)
@@
 		)
 	)
+	(hierarchical_label "CMD{slash}DI"
+		(shape input)
+		(at 127 71.12 0)
+		(effects
+			(font
+				(size 1.27 1.27)
+			)
+			(justify left)
+		)
+	)
 	(hierarchical_label "AV_IN"
 		(shape bidirectional)
@@
 		)
 	)
+	(hierarchical_label "CS{slash}CD"
+		(shape input)
+		(at 166.37 139.7 180)
+		(effects
+			(font
+				(size 1.27 1.27)
+			)
+			(justify right)
+		)
+	)
 	(hierarchical_label "NPN_I2"
 		(shape input)
@@
 		)
 	)
+	(hierarchical_label "DO"
+		(shape input)
+		(at 127 66.04 0)
+		(effects
+			(font
+				(size 1.27 1.27)
+			)
+			(justify left)
+		)
+	)
 	(hierarchical_label "mA_IN"
 		(shape bidirectional)
@@
 		)
 	)
+	(hierarchical_label "DO"
+		(shape input)
+		(at 166.37 142.24 180)
+		(effects
+			(font
+				(size 1.27 1.27)
+			)
+			(justify right)
+		)
+	)
 	(hierarchical_label "VOLTAGE_AOUTPUT"
 		(shape bidirectional)
@@
 		)
 	)
+	(hierarchical_label "CS{slash}CD"
+		(shape input)
+		(at 127 68.58 0)
+		(effects
+			(font
+				(size 1.27 1.27)
+			)
+			(justify left)
+		)
+	)
 	(hierarchical_label "NPN_O2"
 		(shape input)
@@
 			)
 		)
+		(pin "CMD{slash}DI" input
+			(at 125.73 71.12 0)
+			(effects
+				(font
+					(size 1.27 1.27)
+				)
+				(justify right)
+			)
+		)
+		(pin "CS{slash}CD" input
+			(at 125.73 68.58 0)
+			(effects
+				(font
+					(size 1.27 1.27)
+				)
+				(justify right)
+			)
+		)
+		(pin "DO" input
+			(at 125.73 66.04 0)
+			(effects
+				(font
+					(size 1.27 1.27)
+				)
+				(justify right)
+			)
+		)
 		(instances
 			(project "PLC4UNI_Board"
@@
 				)
 			)
+		)
+	)
+	(sheet
+		(at 168.275 133.985)
+		(size 22.225 20.32)
+		(exclude_from_sim no)
+		(in_bom yes)
+		(on_board yes)
+		(dnp no)
+		(fields_autoplaced yes)
+		(stroke
+			(width 0.1524)
+			(type solid)
+		)
+		(fill
+			(color 0 0 0 0.0000)
+		)
+		(property "Sheetname" "SD"
+			(at 168.275 133.2734 0)
+			(effects
+				(font
+					(size 1.27 1.27)
+				)
+				(justify left bottom)
+			)
+		)
+		(property "Sheetfile" "SDC.kicad_sch"
+			(at 168.275 154.8896 0)
+			(effects
+				(font
+					(size 1.27 1.27)
+				)
+				(justify left top)
+			)
+		)
+		(pin "CMD{slash}DI" input
+			(at 168.275 137.16 180)
+			(effects
+				(font
+					(size 1.27 1.27)
+				)
+				(justify left)
+			)
+		)
+		(pin "CS{slash}CD" input
+			(at 168.275 139.7 180)
+			(effects
+				(font
+					(size 1.27 1.27)
+				)
+				(justify left)
+			)
+		)
+		(pin "DO" input
+			(at 168.275 142.24 180)
+			(effects
+				(font
+					(size 1.27 1.27)
+				)
+				(justify left)
+			)
+		)
+		(pin "SCLK" input
+			(at 168.275 144.78 180)
+			(effects
+				(font
+					(size 1.27 1.27)
+				)
+				(justify left)
+			)
+		)
+		(instances
+			(project "PLC4UNI_Board"
+				(path "/3f95a48a-e63f-444a-b104-97d170acd68f"
+					(page "27")
+				)
+			)
