File: PLC4UNI_Board/PNPO.kicad_sch (KiCad schematic)
At the start: 0 parts

Commit message: V1.0.2 PLC4UNI
Parts:
- added Q1: TIP41, Package_TO_SOT_THT:TO-220-3_Vertical, symbol Transistor_BJT:TIP41
- added U11: TLP290, Package_SO:SOP-4_4.4x2.6mm_P1.27mm, symbol Isolator:TLP290
Connections:
- new net: Q1.1 (B), U11.3
- new net GND2: U11.2
- new net PNP_MCO_1: U11.1
- new net PNP_OUT_1: Q1.2 (C), U11.4
- new net VCC: Q1.3 (E)

Commit message: main
Parts:
- removed Q1: TIP41, Package_TO_SOT_THT:TO-220-3_Vertical, symbol Transistor_BJT:TIP41
- added Q9: TIP42, Package_TO_SOT_THT:TO-220-3_Vertical, symbol Transistor_BJT:TIP42
Connections:
- net PNP_OUT_1: now also Q9.2 (C)
- net VCC: now also Q9.3 (E)
- net at U11.3: now also Q9.1 (B)
Changed lines of the file:
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@@
-	(wire
-		(pts
-			(xy 129.54 60.96) (xy 133.35 60.96)
-		)
-		(stroke
-			(width 0)
-			(type default)
-		)
-	)
 	(wire
 		(pts
@@
 	(wire
 		(pts
-			(xy 129.54 71.12) (xy 149.86 71.12)
+			(xy 129.54 60.96) (xy 133.35 60.96)
+		)
+		(stroke
+			(width 0)
+			(type default)
+		)
+	)
+	(wire
+		(pts
+			(xy 137.16 71.12) (xy 129.54 71.12)
 		)
 		(stroke
@@
 	)
 	(symbol
+		(lib_id "Transistor_BJT:TIP42")
+		(at 127 66.04 0)
+		(unit 1)
+		(exclude_from_sim no)
+		(in_bom yes)
+		(on_board yes)
+		(dnp no)
+		(property "Reference" "Q9"
+			(at 132.08 64.7699 0)
+			(effects
+				(font
+					(size 1.27 1.27)
+				)
+				(justify left)
+			)
+		)
+		(property "Value" "TIP42"
+			(at 132.08 67.3099 0)
+			(effects
+				(font
+					(size 1.27 1.27)
+				)
+				(justify left)
+			)
+		)
+		(property "Footprint" "Package_TO_SOT_THT:TO-220-3_Vertical"
+			(at 133.35 67.945 0)
+			(effects
+				(font
+					(size 1.27 1.27)
+					(italic yes)
+				)
+				(justify left)
+				(hide yes)
+			)
+		)
+		(property "Datasheet" "https://www.centralsemi.com/get_document.php?cmp=1&mergetype=pd&mergepath=pd&pdf_id=TIP42.PDF"
+			(at 127 66.04 0)
+			(effects
+				(font
+					(size 1.27 1.27)
+				)
+				(justify left)
+				(hide yes)
+			)
+		)
+		(property "Description" "-6A Ic, -40V Vce, Power PNP Transistor, TO-220"
+			(at 127 66.04 0)
+			(effects
+				(font
+					(size 1.27 1.27)
+				)
+				(hide yes)
+			)
+		)
+		(pin "2"
+		)
+		(pin "3"
+		)
+		(pin "1"
+		)
+		(instances
+			(project ""
+				(path "/3f95a48a-e63f-444a-b104-97d170acd68f/54f02f4d-f252-448d-96ba-66650260df5f"
+					(reference "Q11")
+					(unit 1)
+				)
+				(path "/3f95a48a-e63f-444a-b104-97d170acd68f/9dd420b4-935b-4e1c-80b3-c53481129f98"
+					(reference "Q9")
+					(unit 1)
+				)
+				(path "/3f95a48a-e63f-444a-b104-97d170acd68f/d52f26c0-222f-43e7-a488-474b82d7e3e7"
+					(reference "Q10")
+					(unit 1)
+				)
+			)
+		)
+	)
+	(symbol
 		(lib_id "power:GND1")
 		(at 106.68 68.58 0)
@@
 				(path "/3f95a48a-e63f-444a-b104-97d170acd68f/d52f26c0-222f-43e7-a488-474b82d7e3e7"
 					(reference "#PWR042")
-					(unit 1)
-				)
-			)
-		)
-	)
-	(symbol
-		(lib_id "Transistor_BJT:TIP41")
-		(at 127 66.04 0)
-		(unit 1)
-		(exclude_from_sim no)
-		(in_bom yes)
-		(on_board yes)
-		(dnp no)
-		(fields_autoplaced yes)
-		(property "Reference" "Q1"
-			(at 132.08 64.7699 0)
-			(effects
-				(font
-					(size 1.27 1.27)
-				)
-				(justify left)
-			)
-		)
-		(property "Value" "TIP41"
-			(at 132.08 67.3099 0)
-			(effects
-				(font
-					(size 1.27 1.27)
-				)
-				(justify left)
-			)
-		)
-		(property "Footprint" "Package_TO_SOT_THT:TO-220-3_Vertical"
-			(at 133.35 67.945 0)
-			(effects
-				(font
-					(size 1.27 1.27)
-					(italic yes)
-				)
-				(justify left)
-				(hide yes)
-			)
-		)
-		(property "Datasheet" "https://www.centralsemi.com/get_document.php?cmp=1&mergetype=pd&mergepath=pd&pdf_id=tip41.PDF"
-			(at 127 66.04 0)
-			(effects
-				(font
-					(size 1.27 1.27)
-				)
-				(justify left)
-				(hide yes)
-			)
-		)
-		(property "Description" "6A Ic, 40V Vce, Power NPN Transistor, TO-220"
-			(at 127 66.04 0)
-			(effects
-				(font
-					(size 1.27 1.27)
-				)
-				(hide yes)
-			)
-		)
-		(pin "3"
-		)
-		(pin "1"
-		)
-		(pin "2"
-		)
-		(instances
-			(project ""
-				(path "/3f95a48a-e63f-444a-b104-97d170acd68f/54f02f4d-f252-448d-96ba-66650260df5f"
-					(reference "Q3")
-					(unit 1)
-				)
-				(path "/3f95a48a-e63f-444a-b104-97d170acd68f/9dd420b4-935b-4e1c-80b3-c53481129f98"
-					(reference "Q1")
-					(unit 1)
-				)
-				(path "/3f95a48a-e63f-444a-b104-97d170acd68f/d52f26c0-222f-43e7-a488-474b82d7e3e7"
-					(reference "Q2")
 					(unit 1)
 				)
@@
 	(symbol
 		(lib_id "power:VCC")
-		(at 149.86 71.12 0)
+		(at 137.16 71.12 0)
 		(unit 1)
 		(exclude_from_sim no)
@@
 		(fields_autoplaced yes)
 		(property "Reference" "#PWR038"
-			(at 149.86 74.93 0)
+			(at 137.16 74.93 0)
 			(effects
 				(font
@@
 		)
 		(property "Value" "VCC"
-			(at 149.86 66.04 0)
-			(effects
-				(font
-					(size 1.27 1.27)
-				)
+			(at 139.7 69.8499 0)
+			(effects
+				(font
+					(size 1.27 1.27)
+				)
+				(justify left)
 			)
 		)
 		(property "Footprint" ""
-			(at 149.86 71.12 0)
+			(at 137.16 71.12 0)
 			(effects
 				(font
@@
 		)
 		(property "Datasheet" ""
-			(at 149.86 71.12 0)
+			(at 137.16 71.12 0)
 			(effects
 				(font
@@
 		)
 		(property "Description" "Power symbol creates a global label with name \"VCC\""
-			(at 149.86 71.12 0)
-			(effects
-				(font
+			(at 137.16 71.12 0)
+			(effects
+				(font

Commit message: v.3.0.0
Connections:
- net GND2 renamed GND
Changed lines of the file:
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@@
 			)
 		)
-		(property "Value" "GND2"
+		(property "Value" "GND"
 			(at 106.68 73.66 0)
 			(effects

Commit message: main
Parts:
- Q9: footprint Package_TO_SOT_THT:TO-220-3_Vertical -> Package_TO_SOT_SMD:TO-252-2
Changed lines of the file:
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@@
 			)
 		)
-		(property "Footprint" "Package_TO_SOT_THT:TO-220-3_Vertical"
+		(property "Footprint" "Package_TO_SOT_SMD:TO-252-2"
 			(at 133.35 67.945 0)
 			(effects
