File: PLC4UNI_Board/RLY1.kicad_sch (KiCad schematic)
At the start: 5 parts, among them K2 G5Q-1, Q8 TIP41, U18 TLP290

Commit message: main
Parts:
- Q8: footprint Package_TO_SOT_THT:TO-220-3_Vertical -> Package_TO_SOT_SMD:TO-252-2
Changed lines of the file:
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@@
 			)
 		)
-		(property "Footprint" "Package_TO_SOT_THT:TO-220-3_Vertical"
+		(property "Footprint" "Package_TO_SOT_SMD:TO-252-2"
 			(at 121.92 111.125 0)
 			(effects
