File: PLC4UNI_Board/mA_INTERFAZ.kicad_sch (KiCad schematic)
At the start: 18 parts, among them T1 IRF9310TRPBF

Commit message: main
Parts:
- D7: footprint Diode_THT:D_DO-41_SOD81_P10.16mm_Horizontal -> Diode_SMD:D_0603_1608Metric_Pad1.05x0.95mm_HandSolder
Changed lines of the file:
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@@
 			)
 		)
-		(property "Footprint" "Diode_THT:D_DO-41_SOD81_P10.16mm_Horizontal"
+		(property "Footprint" "Diode_SMD:D_0603_1608Metric_Pad1.05x0.95mm_HandSolder"
 			(at 204.47 65.405 0)
 			(effects
