File: PLC4UNI_Board/PSU_sch.kicad_sch (KiCad schematic)
At the start: 9 parts, among them U2 AP63203WU

Commit message: V1.0.2 PLC4UNI
Parts:
- renumbered C3 to C2, C4 to C3, C2 to C4, L2 to L1, R24 to R2, R25 to R3
Changed lines of the file:
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@@
 		(dnp no)
 		(fields_autoplaced yes)
-		(property "Reference" "#PWR049"
+		(property "Reference" "#PWR014"
 			(at 154.94 107.95 0)
 			(effects
@@
 		(instances
 			(project "PLC4UNI_Board"
-				(path "/3f95a48a-e63f-444a-b104-97d170acd68f/331a08dd-fee0-4544-a181-684d5445d70e/e5218d9c-20b6-4436-adf7-9f480a59cb72"
-					(reference "#PWR049")
+				(path "/3f95a48a-e63f-444a-b104-97d170acd68f/19dcce3c-991e-4eb9-8758-67e295a30a53"
+					(reference "#PWR014")
 					(unit 1)
 				)
@@
 		(dnp no)
 		(fields_autoplaced yes)
-		(property "Reference" "R25"
+		(property "Reference" "R3"
 			(at 157.48 95.2499 0)
 			(effects
@@
 		(instances
 			(project "PLC4UNI_Board"
-				(path "/3f95a48a-e63f-444a-b104-97d170acd68f/331a08dd-fee0-4544-a181-684d5445d70e/e5218d9c-20b6-4436-adf7-9f480a59cb72"
-					(reference "R25")
+				(path "/3f95a48a-e63f-444a-b104-97d170acd68f/19dcce3c-991e-4eb9-8758-67e295a30a53"
+					(reference "R3")
 					(unit 1)
 				)
@@
 		(dnp no)
 		(fields_autoplaced yes)
-		(property "Reference" "#PWR011"
+		(property "Reference" "#PWR015"
 			(at 163.83 72.39 0)
 			(effects
@@
 		(instances
 			(project "PLC4UNI_Board"
-				(path "/3f95a48a-e63f-444a-b104-97d170acd68f/331a08dd-fee0-4544-a181-684d5445d70e/e5218d9c-20b6-4436-adf7-9f480a59cb72"
-					(reference "#PWR011")
+				(path "/3f95a48a-e63f-444a-b104-97d170acd68f/19dcce3c-991e-4eb9-8758-67e295a30a53"
+					(reference "#PWR015")
 					(unit 1)
 				)
@@
 		(dnp no)
 		(fields_autoplaced yes)
-		(property "Reference" "#PWR050"
+		(property "Reference" "#PWR048"
 			(at 180.34 88.9 0)
 			(effects
@@
 		(instances
 			(project "PLC4UNI_Board"
-				(path "/3f95a48a-e63f-444a-b104-97d170acd68f/331a08dd-fee0-4544-a181-684d5445d70e/e5218d9c-20b6-4436-adf7-9f480a59cb72"
-					(reference "#PWR050")
+				(path "/3f95a48a-e63f-444a-b104-97d170acd68f/19dcce3c-991e-4eb9-8758-67e295a30a53"
+					(reference "#PWR048")
 					(unit 1)
 				)
@@
 		(dnp no)
 		(fields_autoplaced yes)
-		(property "Reference" "#PWR048"
+		(property "Reference" "#PWR013"
 			(at 114.3 106.68 0)
 			(effects
@@
 		(instances
 			(project "PLC4UNI_Board"
-				(path "/3f95a48a-e63f-444a-b104-97d170acd68f/331a08dd-fee0-4544-a181-684d5445d70e/e5218d9c-20b6-4436-adf7-9f480a59cb72"
-					(reference "#PWR048")
+				(path "/3f95a48a-e63f-444a-b104-97d170acd68f/19dcce3c-991e-4eb9-8758-67e295a30a53"
+					(reference "#PWR013")
 					(unit 1)
 				)
@@
 		(dnp no)
 		(fields_autoplaced yes)
-		(property "Reference" "C3"
+		(property "Reference" "C2"
 			(at 95.25 92.7099 0)
 			(effects
@@
 		(instances
 			(project "PLC4UNI_Board"
-				(path "/3f95a48a-e63f-444a-b104-97d170acd68f/331a08dd-fee0-4544-a181-684d5445d70e/e5218d9c-20b6-4436-adf7-9f480a59cb72"
-					(reference "C3")
+				(path "/3f95a48a-e63f-444a-b104-97d170acd68f/19dcce3c-991e-4eb9-8758-67e295a30a53"
+					(reference "C2")
 					(unit 1)
 				)
@@
 		(instances
 			(project "PLC4UNI_Board"
-				(path "/3f95a48a-e63f-444a-b104-97d170acd68f/331a08dd-fee0-4544-a181-684d5445d70e/e5218d9c-20b6-4436-adf7-9f480a59cb72"
+				(path "/3f95a48a-e63f-444a-b104-97d170acd68f/19dcce3c-991e-4eb9-8758-67e295a30a53"
 					(reference "C6")
 					(unit 1)
@@
 		(instances
 			(project "PLC4UNI_Board"
-				(path "/3f95a48a-e63f-444a-b104-97d170acd68f/331a08dd-fee0-4544-a181-684d5445d70e/e5218d9c-20b6-4436-adf7-9f480a59cb72"
+				(path "/3f95a48a-e63f-444a-b104-97d170acd68f/19dcce3c-991e-4eb9-8758-67e295a30a53"
 					(reference "C5")
 					(unit 1)
@@
 		(dnp no)
 		(fields_autoplaced yes)
-		(property "Reference" "R24"
+		(property "Reference" "R2"
 			(at 157.48 86.3599 0)
 			(effects
@@
 		(instances
 			(project "PLC4UNI_Board"
-				(path "/3f95a48a-e63f-444a-b104-97d170acd68f/331a08dd-fee0-4544-a181-684d5445d70e/e5218d9c-20b6-4436-adf7-9f480a59cb72"
-					(reference "R24")
+				(path "/3f95a48a-e63f-444a-b104-97d170acd68f/19dcce3c-991e-4eb9-8758-67e295a30a53"
+					(reference "R2")
 					(unit 1)
 				)
@@
 		(dnp no)
 		(fields_autoplaced yes)
-		(property "Reference" "C4"
+		(property "Reference" "C3"
 			(at 134.62 76.2 90)
 			(effects
@@
 		(instances
 			(project "PLC4UNI_Board"
-				(path "/3f95a48a-e63f-444a-b104-97d170acd68f/331a08dd-fee0-4544-a181-684d5445d70e/e5218d9c-20b6-4436-adf7-9f480a59cb72"
-					(reference "C4")
+				(path "/3f95a48a-e63f-444a-b104-97d170acd68f/19dcce3c-991e-4eb9-8758-67e295a30a53"
+					(reference "C3")
 					(unit 1)
 				)
@@
 		(dnp no)
 		(fields_autoplaced yes)
-		(property "Reference" "C2"
+		(property "Reference" "C4"
 			(at 147.32 86.3599 0)
 			(effects
@@
 		(instances
 			(project "PLC4UNI_Board"
-				(path "/3f95a48a-e63f-444a-b104-97d170acd68f/331a08dd-fee0-4544-a181-684d5445d70e/e5218d9c-20b6-4436-adf7-9f480a59cb72"
-					(reference "C2")
+				(path "/3f95a48a-e63f-444a-b104-97d170acd68f/19dcce3c-991e-4eb9-8758-67e295a30a53"
+					(reference "C4")
 					(unit 1)
 				)
@@
 		(dnp no)
 		(fields_autoplaced yes)
-		(property "Reference" "L2"
+		(property "Reference" "L1"
 			(at 128.27 74.9299 0)
 			(effects
@@
 		(instances
 			(project "PLC4UNI_Board"
-				(path "/3f95a48a-e63f-444a-b104-97d170acd68f/331a08dd-fee0-4544-a181-684d5445d70e/e5218d9c-20b6-4436-adf7-9f480a59cb72"
-					(reference "L2")
+				(path "/3f95a48a-e63f-444a-b104-97d170acd68f/19dcce3c-991e-4eb9-8758-67e295a30a53"
+					(reference "L1")
 					(unit 1)
 				)
@@
 		(dnp no)
 		(fields_autoplaced yes)
-		(property "Reference" "#PWR051"
+		(property "Reference" "#PWR047"
 			(at 168.91 88.9 0)
 			(effects
@@
 		(instances
 			(project "PLC4UNI_Board"
-				(path "/3f95a48a-e63f-444a-b104-97d170acd68f/331a08dd-fee0-4544-a181-684d5445d70e/e5218d9c-20b6-4436-adf7-9f480a59cb72"
-					(reference "#PWR051")
+				(path "/3f95a48a-e63f-444a-b104-97d170acd68f/19dcce3c-991e-4eb9-8758-67e295a30a53"
+					(reference "#PWR047")
 					(unit 1)
 				)
@@
 		(instances
 			(project "PLC4UNI_Board"
-				(path "/3f95a48a-e63f-444a-b104-97d170acd68f/331a08dd-fee0-4544-a181-684d5445d70e/e5218d9c-20b6-4436-adf7-9f480a59cb72"
+				(path "/3f95a48a-e63f-444a-b104-97d170acd68f/19dcce3c-991e-4eb9-8758-67e295a30a53"
 					(reference "U2")
 					(unit 1)
@@
 		(dnp no)
 		(fields_autoplaced yes)
-		(property "Reference" "#PWR047"
+		(property "Reference" "#PWR012"
 			(at 91.44 106.68 0)
 			(effects
@@
 		(instances
 			(project "PLC4UNI_Board"
-				(path "/3f95a48a-e63f-444a-b104-97d170acd68f/331a08dd-fee0-4544-a181-684d5445d70e/e5218d9c-20b6-4436-adf7-9f480a59cb72"
-					(reference "#PWR047")
+				(path "/3f95a48a-e63f-444a-b104-97d170acd68f/19dcce3c-991e-4eb9-8758-67e295a30a53"
+					(reference "#PWR012")
 					(unit 1)
 				)
@@
 		(dnp no)
 		(fields_autoplaced yes)
-		(property "Reference" "#PWR012"
+		(property "Reference" "#PWR011"
 			(at 91.44 87.63 0)
 			(effects
@@
 		(instances
 			(project "PLC4UNI_Board"
-				(path "/3f95a48a-e63f-444a-b104-97d170acd68f/331a08dd-fee0-4544-a181-684d5445d70e/e5218d9c-20b6-4436-adf7-9f480a59cb72"
-					(reference "#PWR012")
-					(unit 1)
-				)
+				(path "/3f95a48a-e63f-444a-b104-97d170acd68f/19dcce3c-991e-4eb9-8758-67e295a30a53"
+					(reference "#PWR011")
+					(unit 1)
+				)

Commit message: main
Parts:
- C2: footprint PCM_Capacitor_SMD_AKL:C_1206_3216Metric -> Capacitor_SMD:C_1206_3216Metric
- C3: footprint PCM_Capacitor_SMD_AKL:C_0603_1608Metric -> Capacitor_SMD:C_0201_0603Metric
- C4: footprint PCM_Capacitor_SMD_AKL:C_1206_3216Metric -> Capacitor_SMD:C_1206_3216Metric_Pad1.33x1.80mm_HandSolder
- C5, C6: footprint PCM_Capacitor_SMD_AKL:C_0805_2012Metric -> Capacitor_SMD:C_0805_2012Metric_Pad1.18x1.45mm_HandSolder
- R2, R3: footprint (none) -> Resistor_SMD:R_0201_0603Metric
Changed lines of the file:
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@@
 			)
 		)
-		(property "Footprint" ""
+		(property "Footprint" "Resistor_SMD:R_0201_0603Metric"
 			(at 155.956 96.774 90)
 			(effects
@@
 			)
 		)
-		(property "Footprint" "PCM_Capacitor_SMD_AKL:C_1206_3216Metric"
+		(property "Footprint" "Capacitor_SMD:C_1206_3216Metric"
 			(at 92.4052 99.06 0)
 			(effects
@@
 			)
 		)
-		(property "Footprint" "PCM_Capacitor_SMD_AKL:C_0805_2012Metric"
+		(property "Footprint" "Capacitor_SMD:C_0805_2012Metric_Pad1.18x1.45mm_HandSolder"
 			(at 181.3052 82.55 0)
 			(effects
@@
 			)
 		)
-		(property "Footprint" "PCM_Capacitor_SMD_AKL:C_0805_2012Metric"
+		(property "Footprint" "Capacitor_SMD:C_0805_2012Metric_Pad1.18x1.45mm_HandSolder"
 			(at 169.8752 82.55 0)
 			(effects
@@
 			)
 		)
-		(property "Footprint" ""
+		(property "Footprint" "Resistor_SMD:R_0201_0603Metric"
 			(at 155.956 87.884 90)
 			(effects
@@
 			)
 		)
-		(property "Footprint" "PCM_Capacitor_SMD_AKL:C_0603_1608Metric"
+		(property "Footprint" "Capacitor_SMD:C_0201_0603Metric"
 			(at 138.43 85.3948 0)
 			(effects
@@
 			)
 		)
-		(property "Footprint" "PCM_Capacitor_SMD_AKL:C_1206_3216Metric"
+		(property "Footprint" "Capacitor_SMD:C_1206_3216Metric_Pad1.33x1.80mm_HandSolder"
 			(at 144.4752 91.44 0)
 			(effects
@@
 		(on_board yes)
 		(dnp no)
-		(fields_autoplaced yes)
 		(property "Reference" "L1"
 			(at 128.27 74.9299 0)
@@
 		)
 		(property "Display" "6.8uH"
-			(at 128.27 77.4699 0)
+			(at 120.396 75.438 0)
 			(effects
 				(font
@@
 		)
 		(property "Display 2" "1.6A"
-			(at 128.27 80.0099 0)
-			(effects
-				(font
+			(at 120.904 77.978 0)
+			(effects
+				(font

Commit message: main
Parts:
- added D10: 1N5819, Diode_THT:D_DO-41_SOD81_P10.16mm_Horizontal, symbol Diode:1N5819
- C3: footprint Capacitor_SMD:C_0201_0603Metric -> Resistor_SMD:R_0805_2012Metric
- C4: value 22uF -> 100pf; footprint Capacitor_SMD:C_1206_3216Metric_Pad1.33x1.80mm_HandSolder -> Resistor_SMD:R_0805_2012Metric
- L1: footprint Inductor_SMD:L_APV_ANR6028 -> Inductor_SMD:L_Changjiang_FNR5040S
- R2: value R_US -> 30,9k; footprint Resistor_SMD:R_0201_0603Metric -> Resistor_SMD:R_0805_2012Metric
- R3: value R_US -> 62k
Connections:
- net VCC: now also D10.2 (A); no longer C2.1, U2.2 (EN), U2.3 (IN)
- new net 5vusb: C2.1, D10.1 (K), U2.2 (EN), U2.3 (IN)
Changed lines of the file:
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@@
 	(paper "A4")
+	(junction
+		(at 91.44 90.17)
+		(diameter 0)
+		(color 0 0 0 0)
+	)
+	(junction
+		(at 168.91 74.93)
+		(diameter 0)
+		(color 0 0 0 0)
+	)
+	(junction
+		(at 165.1 74.93)
+		(diameter 0)
+		(color 0 0 0 0)
+	)
+	(junction
+		(at 154.94 74.93)
+		(diameter 0)
+		(color 0 0 0 0)
+	)
+	(junction
+		(at 154.94 92.71)
+		(diameter 0)
+		(color 0 0 0 0)
+	)
 	(junction
 		(at 91.44 91.44)
@@
 	)
 	(junction
-		(at 168.91 74.93)
-		(diameter 0)
-		(color 0 0 0 0)
-	)
-	(junction
-		(at 165.1 74.93)
-		(diameter 0)
-		(color 0 0 0 0)
-	)
-	(junction
-		(at 154.94 74.93)
-		(diameter 0)
-		(color 0 0 0 0)
-	)
-	(junction
-		(at 154.94 92.71)
-		(diameter 0)
-		(color 0 0 0 0)
-	)
-	(junction
 		(at 143.51 92.71)
 		(diameter 0)
@@
 	(wire
 		(pts
+			(xy 91.44 87.63) (xy 91.44 90.17)
+		)
+		(stroke
+			(width 0)
+			(type default)
+		)
+	)
+	(wire
+		(pts
 			(xy 165.1 68.58) (xy 165.1 74.93)
 		)
@@
 	(wire
 		(pts
+			(xy 82.55 90.17) (xy 91.44 90.17)
+		)
+		(stroke
+			(width 0)
+			(type default)
+		)
+	)
+	(wire
+		(pts
 			(xy 124.46 90.17) (xy 138.43 90.17)
 		)
@@
 	(wire
 		(pts
+			(xy 91.44 90.17) (xy 91.44 91.44)
+		)
+		(stroke
+			(width 0)
+			(type default)
+		)
+	)
+	(wire
+		(pts
 			(xy 154.94 73.66) (xy 143.51 73.66)
 		)
@@
 	(wire
 		(pts
-			(xy 91.44 83.82) (xy 91.44 91.44)
-		)
-		(stroke
-			(width 0)
-			(type default)
-		)
-	)
-	(wire
-		(pts
 			(xy 165.1 74.93) (xy 168.91 74.93)
 		)
@@
 	(wire
 		(pts
+			(xy 91.44 78.74) (xy 91.44 80.01)
+		)
+		(stroke
+			(width 0)
+			(type default)
+		)
+	)
+	(wire
+		(pts
 			(xy 163.83 68.58) (xy 165.1 68.58)
 		)
@@
 	(wire
 		(pts
-			(xy 91.44 99.06) (xy 91.44 100.33)
-		)
-		(stroke
-			(width 0)
-			(type default)
+			(xy 91.44 99.06) (xy 91.44 102.87)
+		)
+		(stroke
+			(width 0)
+			(type default)
+		)
+	)
+	(hierarchical_label "5vusb"
+		(shape input)
+		(at 82.55 90.17 180)
+		(effects
+			(font
+				(size 1.27 1.27)
+			)
+			(justify right)
 		)
 	)
@@
 			)
 		)
-		(property "Value" "R_US"
+		(property "Value" "62k"
 			(at 157.48 97.7899 0)
 			(effects
@@
 	)
 	(symbol
+		(lib_id "Diode:1N5819")
+		(at 91.44 83.82 90)
+		(unit 1)
+		(exclude_from_sim no)
+		(in_bom yes)
+		(on_board yes)
+		(dnp no)
+		(property "Reference" "D10"
+			(at 83.82 81.534 90)
+			(effects
+				(font
+					(size 1.27 1.27)
+				)
+				(justify right)
+			)
+		)
+		(property "Value" "1N5819"
+			(at 81.788 83.82 90)
+			(effects
+				(font
+					(size 1.27 1.27)
+				)
+				(justify right)
+			)
+		)
+		(property "Footprint" "Diode_THT:D_DO-41_SOD81_P10.16mm_Horizontal"
+			(at 95.885 83.82 0)
+			(effects
+				(font
+					(size 1.27 1.27)
+				)
+				(hide yes)
+			)
+		)
+		(property "Datasheet" "http://www.vishay.com/docs/88525/1n5817.pdf"
+			(at 91.44 83.82 0)
+			(effects
+				(font
+					(size 1.27 1.27)
+				)
+				(hide yes)
+			)
+		)
+		(property "Description" "40V 1A Schottky Barrier Rectifier Diode, DO-41"
+			(at 91.44 83.82 0)
+			(effects
+				(font
+					(size 1.27 1.27)
+				)
+				(hide yes)
+			)
+		)
+		(pin "2"
+		)
+		(pin "1"
+		)
+		(instances
+			(project ""
+				(path "/3f95a48a-e63f-444a-b104-97d170acd68f/19dcce3c-991e-4eb9-8758-67e295a30a53"
+					(reference "D10")
+					(unit 1)
+				)
+			)
+		)
+	)
+	(symbol
 		(lib_id "PCM_Capacitor_AKL:C_0805")
 		(at 168.91 78.74 0)
@@
 			)
 		)
-		(property "Value" "R_US"
+		(property "Value" "30,9k"
 			(at 157.48 88.8999 0)
 			(effects
@@
 			)
 		)
-		(property "Footprint" "Resistor_SMD:R_0201_0603Metric"
+		(property "Footprint" "Resistor_SMD:R_0805_2012Metric"
 			(at 155.956 87.884 90)
 			(effects
@@
 			)
 		)
-		(property "Footprint" "Capacitor_SMD:C_0201_0603Metric"
+		(property "Footprint" "Resistor_SMD:R_0805_2012Metric"
 			(at 138.43 85.3948 0)
 			(effects
@@
 		(fields_autoplaced yes)
 		(property "Reference" "C4"
-			(at 147.32 86.3599 0)
-			(effects
-				(font
-					(size 1.27 1.27)
-				)
-				(justify left)
-			)
-		)
-		(property "Value" "22uF"
-			(at 147.32 88.8999 0)
-			(effects
-				(font
-					(size 1.27 1.27)
-				)
-				(justify left)
-			)
-		)
-		(property "Footprint" "Capacitor_SMD:C_1206_3216Metric_Pad1.33x1.80mm_HandSolder"
+			(at 147.32 85.0899 0)
+			(effects
+				(font
+					(size 1.27 1.27)
+				)
+				(justify left)
+			)
+		)
+		(property "Value" "100pf"
+			(at 147.32 87.6299 0)
+			(effects
+				(font
+					(size 1.27 1.27)
+				)
+				(justify left)
+			)
+		)
+		(property "Footprint" "Resistor_SMD:R_0805_2012Metric"
 			(at 144.4752 91.44 0)
 			(effects
@@
 		)
 		(property "volt" "10v"
-			(at 143.51 87.63 0)
-			(effects
-				(font
-					(size 1.27 1.27)
-				)
+			(at 147.32 90.1699 0)
+			(effects
+				(font
+					(size 1.27 1.27)
+				)
+				(justify left)
 			)
 		)
@@
 			)
 		)
-		(property "Footprint" "Inductor_SMD:L_APV_ANR6028"
+		(property "Footprint" "Inductor_SMD:L_Changjiang_FNR5040S"
 			(at 127 90.17 0)
 			(effects
@@
 	(symbol
 		(lib_id "power:GND")
-		(at 91.44 100.33 0)
+		(at 91.44 102.87 0)
 		(unit 1)
 		(exclude_from_sim no)
@@
 		(fields_autoplaced yes)
 		(property "Reference" "#PWR012"
-			(at 91.44 106.68 0)
+			(at 91.44 109.22 0)
 			(effects
 				(font
@@
 		)
 		(property "Value" "GND"
-			(at 91.44 105.41 0)
+			(at 91.44 107.95 0)
 			(effects
 				(font
@@
 		)
 		(property "Footprint" ""
-			(at 91.44 100.33 0)
+			(at 91.44 102.87 0)
 			(effects
 				(font
@@
 		)
 		(property "Datasheet" ""
-			(at 91.44 100.33 0)
+			(at 91.44 102.87 0)
 			(effects
 				(font
@@
 		)
 		(property "Description" "Power symbol creates a global label with name \"GND\" , ground"
-			(at 91.44 100.33 0)
+			(at 91.44 102.87 0)
 			(effects
 				(font
@@
 	(symbol
 		(lib_id "power:VCC")
-		(at 91.44 83.82 0)
+		(at 91.44 78.74 0)
 		(unit 1)
 		(exclude_from_sim no)
@@
 		(fields_autoplaced yes)
 		(property "Reference" "#PWR011"
-			(at 91.44 87.63 0)
+			(at 91.44 82.55 0)
 			(effects
 				(font
@@
 		)
 		(property "Value" "VCC"
+			(at 91.44 73.66 0)
+			(effects
+				(font
+					(size 1.27 1.27)
+				)
+			)
+		)
+		(property "Footprint" ""
 			(at 91.44 78.74 0)
 			(effects
@@
 					(size 1.27 1.27)
 				)
-			)
-		)
-		(property "Footprint" ""
-			(at 91.44 83.82 0)
-			(effects
-				(font
-					(size 1.27 1.27)
-				)
 				(hide yes)
 			)
 		)
 		(property "Datasheet" ""
-			(at 91.44 83.82 0)
+			(at 91.44 78.74 0)
 			(effects
 				(font
@@
 		)
 		(property "Description" "Power symbol creates a global label with name \"VCC\""
-			(at 91.44 83.82 0)
-			(effects
-				(font
+			(at 91.44 78.74 0)
+			(effects
+				(font

Commit message: main
Parts:
- D10: footprint Diode_THT:D_DO-41_SOD81_P10.16mm_Horizontal -> Diode_SMD:D_0603_1608Metric_Pad1.05x0.95mm_HandSolder
Changed lines of the file:
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@@
 			)
 		)
-		(property "Footprint" "Diode_THT:D_DO-41_SOD81_P10.16mm_Horizontal"
+		(property "Footprint" "Diode_SMD:D_0603_1608Metric_Pad1.05x0.95mm_HandSolder"
 			(at 95.885 83.82 0)
 			(effects
